Commit message: Gazebo

File: src/scene/urdf/sim-robot.xacro (robot description, xacro)
@@ -9,4 +9,27 @@
   <xacro:property name="transparency" value="0.8" />
   <xacro:property name="PI" value="3.1415926535" />
+  <xacro:property name="foot_mass" value="0.001" />
+  <xacro:property name="base_mass" value="20.0" />
+  <xacro:property name="lidar_mass" value="5.0" />
+  <xacro:property name="imu_mass" value="1.0" />
+  <xacro:property name="camera_mass" value="1.0" />
+  <xacro:macro name="cylinder_inertial_matrix" params="m r h">
+    <inertial>
+      <mass value="${m}" />
+      <inertia ixx="${m*(3*r*r+h*h)/12}" ixy="0" ixz="0" iyy="${m*(3*r*r+h*h)/12}" iyz="0" izz="${m*r*r/2}" />
+    </inertial>
+  </xacro:macro>
+  <xacro:macro name="box_inertial_matrix" params="m l w h">
+    <inertial>
+      <mass value="${m}" />
+      <inertia ixx="${m*(h*h + l*l)/12}" ixy="0" ixz="0" iyy="${m*(w*w + l*l)/12}" iyz="0" izz="${m*(w*w + h*h)/12}" />
+    </inertial>
+  </xacro:macro>
+  <xacro:macro name="sphere_inertial_matrix" params="m r">
+    <inertial>
+      <mass value="${m}" />
+      <inertia ixx="${2*m*r*r/5}" ixy="0" ixz="0" iyy="${2*m*r*r/5}" iyz="0" izz="${2*m*r*r/5}" />
+    </inertial>
+  </xacro:macro>
   <!-- foot base link -->
   <link name="base_footprint">
@@ -19,4 +42,11 @@
       </material>
     </visual>
+    <collision>
+      <geometry>
+        <box size="${foot_box_size} ${foot_box_size} ${foot_box_size}" />
+      </geometry>
+      <origin xyz="0.0 0.0 0.0" rpy="0.0 0.0 0.0" />
+    </collision>
+    <xacro:box_inertial_matrix m="${foot_mass}" l="${foot_box_size}" w="${foot_box_size}" h="${foot_box_size}" />
   </link>
   <!-- base link -->
@@ -30,4 +60,11 @@
       </material>
     </visual>
+    <collision>
+      <geometry>
+        <box size="${base_box_size} ${base_box_size} ${base_box_size}" />
+      </geometry>
+      <origin xyz="0.0 0.0 0.0" rpy="0.0 0.0 0.0" />
+    </collision>
+    <xacro:box_inertial_matrix m="${base_mass}" l="${base_box_size}" w="${base_box_size}" h="${base_box_size}" />
   </link>
   <!-- joint -->
@@ -49,4 +86,11 @@
       </material>
     </visual>
+    <collision>
+      <geometry>
+        <cylinder radius="${lidar_cylinder_radius}" length="${lidar_cylinder_length}" />
+      </geometry>
+      <origin xyz="0.0 0.0 0.0" rpy="0.0 0.0 0.0" />
+    </collision>
+    <xacro:cylinder_inertial_matrix m="${lidar_mass}" r="${lidar_cylinder_radius}" h="${lidar_cylinder_length}" />
   </link>
   <!-- joint -->
@@ -68,4 +112,11 @@
       </material>
     </visual>
+    <collision>
+      <geometry>
+        <box size="${imu_box_size} ${imu_box_size} ${imu_box_size}" />
+      </geometry>
+      <origin xyz="0.0 0.0 0.0" rpy="0.0 0.0 0.0" />
+    </collision>
+    <xacro:box_inertial_matrix m="${imu_mass}" l="${imu_box_size}" w="${imu_box_size}" h="${imu_box_size}" />
   </link>
   <!-- joint -->
@@ -87,4 +138,11 @@
       </material>
     </visual>
+    <collision>
+      <geometry>
+        <cylinder radius="${camera_cylinder_radius}" length="${camera_cylinder_length}" />
+      </geometry>
+      <origin xyz="0.0 0.0 0.0" rpy="0.0 0.0 0.0" />
+    </collision>
+    <xacro:cylinder_inertial_matrix m="${camera_mass}" r="${camera_cylinder_radius}" h="${camera_cylinder_length}" />
   </link>
   <!-- joint -->
@@ -95,3 +153,18 @@
     <axis xyz="0.0 0.0 1.0" />
   </joint>
+  <gazebo reference="base_footprint">
+    <material>Gazebo/Black</material>
+  </gazebo>
+  <gazebo reference="base_link">
+    <material>Gazebo/White</material>
+  </gazebo>
+  <gazebo reference="lidar">
+    <material>Gazebo/Red</material>
+  </gazebo>
+  <gazebo reference="imu">
+    <material>Gazebo/Green</material>
+  </gazebo>
+  <gazebo reference="camera">
+    <material>Gazebo/Blue</material>
+  </gazebo>
 </robot>

Commit message: split xacro

File: src/scene/urdf/sim-robot.xacro (robot description, xacro)
@@ -50,4 +50,7 @@
     <xacro:box_inertial_matrix m="${foot_mass}" l="${foot_box_size}" w="${foot_box_size}" h="${foot_box_size}" />
   </link>
+  <gazebo reference="base_footprint">
+    <material>Gazebo/Black</material>
+  </gazebo>
   <!-- base link -->
   <link name="base_link">
@@ -68,4 +71,7 @@
     <xacro:box_inertial_matrix m="${base_mass}" l="${base_box_size}" w="${base_box_size}" h="${base_box_size}" />
   </link>
+  <gazebo reference="base_link">
+    <material>Gazebo/White</material>
+  </gazebo>
   <!-- joint -->
   <joint name="base_to_foot" type="fixed">
@@ -75,96 +81,6 @@
     <axis xyz="0.0 0.0 1.0" />
   </joint>
-  <!-- lidar -->
-  <link name="lidar">
-    <visual>
-      <geometry>
-        <cylinder radius="${lidar_cylinder_radius}" length="${lidar_cylinder_length}" />
-      </geometry>
-      <origin xyz="0.0 0.0 0.0" rpy="0.0 0.0 0.0" />
-      <material name="red">
-        <color rgba="1.0 0.0 0.0 ${transparency}" />
-      </material>
-    </visual>
-    <collision>
-      <geometry>
-        <cylinder radius="${lidar_cylinder_radius}" length="${lidar_cylinder_length}" />
-      </geometry>
-      <origin xyz="0.0 0.0 0.0" rpy="0.0 0.0 0.0" />
-    </collision>
-    <xacro:cylinder_inertial_matrix m="${lidar_mass}" r="${lidar_cylinder_radius}" h="${lidar_cylinder_length}" />
-  </link>
-  <!-- joint -->
-  <joint name="lidar_to_base_link" type="fixed">
-    <parent link="base_link" />
-    <child link="lidar" />
-    <origin xyz="0.0 0.0 ${base_box_size * 0.5 + lidar_cylinder_length * 0.5}" rpy="0.0 0.0 0.0" />
-    <axis xyz="0.0 0.0 1.0" />
-  </joint>
-  <!-- imu -->
-  <link name="imu">
-    <visual>
-      <geometry>
-        <box size="${imu_box_size} ${imu_box_size} ${imu_box_size}" />
-      </geometry>
-      <origin xyz="0.0 0.0 0.0" rpy="0.0 0.0 0.0" />
-      <material name="green">
-        <color rgba="0.0 1.0 0.0 ${transparency}" />
-      </material>
-    </visual>
-    <collision>
-      <geometry>
-        <box size="${imu_box_size} ${imu_box_size} ${imu_box_size}" />
-      </geometry>
-      <origin xyz="0.0 0.0 0.0" rpy="0.0 0.0 0.0" />
-    </collision>
-    <xacro:box_inertial_matrix m="${imu_mass}" l="${imu_box_size}" w="${imu_box_size}" h="${imu_box_size}" />
-  </link>
-  <!-- joint -->
-  <joint name="imu_to_base_link" type="fixed">
-    <parent link="base_link" />
-    <child link="imu" />
-    <origin xyz="${base_box_size * 0.5 + imu_box_size * 0.5} 0.0 0.0" rpy="${PI} 0.0 0.0" />
-    <axis xyz="0.0 0.0 1.0" />
-  </joint>
-  <!-- camera -->
-  <link name="camera">
-    <visual>
-      <geometry>
-        <cylinder radius="${camera_cylinder_radius}" length="${camera_cylinder_length}" />
-      </geometry>
-      <origin xyz="0.0 0.0 0.0" rpy="0.0 0.0 0.0" />
-      <material name="blue">
-        <color rgba="0.0 0.0 1.0 ${transparency}" />
-      </material>
-    </visual>
-    <collision>
-      <geometry>
-        <cylinder radius="${camera_cylinder_radius}" length="${camera_cylinder_length}" />
-      </geometry>
-      <origin xyz="0.0 0.0 0.0" rpy="0.0 0.0 0.0" />
-    </collision>
-    <xacro:cylinder_inertial_matrix m="${camera_mass}" r="${camera_cylinder_radius}" h="${camera_cylinder_length}" />
-  </link>
-  <!-- joint -->
-  <joint name="camera_to_base_link" type="fixed">
-    <parent link="base_link" />
-    <child link="camera" />
-    <origin xyz="0.0 ${base_box_size * 0.5 + camera_cylinder_length * 0.5} 0.0" rpy="${-PI * 0.5} 0.0 0.0" />
-    <axis xyz="0.0 0.0 1.0" />
-  </joint>
-  <gazebo reference="base_footprint">
-    <material>Gazebo/Black</material>
-  </gazebo>
-  <gazebo reference="base_link">
-    <material>Gazebo/White</material>
-  </gazebo>
-  <gazebo reference="lidar">
-    <material>Gazebo/Red</material>
-  </gazebo>
-  <gazebo reference="imu">
-    <material>Gazebo/Green</material>
-  </gazebo>
-  <gazebo reference="camera">
-    <material>Gazebo/Blue</material>
-  </gazebo>
+  <xacro:include filename="lidar.xacro" />
+  <xacro:include filename="imu.xacro" />
+  <xacro:include filename="camera.xacro" />
 </robot>

Commit message: split xacro macro

File: src/scene/urdf/sim-robot.xacro (robot description, xacro)
@@ -14,22 +14,5 @@
   <xacro:property name="imu_mass" value="1.0" />
   <xacro:property name="camera_mass" value="1.0" />
-  <xacro:macro name="cylinder_inertial_matrix" params="m r h">
-    <inertial>
-      <mass value="${m}" />
-      <inertia ixx="${m*(3*r*r+h*h)/12}" ixy="0" ixz="0" iyy="${m*(3*r*r+h*h)/12}" iyz="0" izz="${m*r*r/2}" />
-    </inertial>
-  </xacro:macro>
-  <xacro:macro name="box_inertial_matrix" params="m l w h">
-    <inertial>
-      <mass value="${m}" />
-      <inertia ixx="${m*(h*h + l*l)/12}" ixy="0" ixz="0" iyy="${m*(w*w + l*l)/12}" iyz="0" izz="${m*(w*w + h*h)/12}" />
-    </inertial>
-  </xacro:macro>
-  <xacro:macro name="sphere_inertial_matrix" params="m r">
-    <inertial>
-      <mass value="${m}" />
-      <inertia ixx="${2*m*r*r/5}" ixy="0" ixz="0" iyy="${2*m*r*r/5}" iyz="0" izz="${2*m*r*r/5}" />
-    </inertial>
-  </xacro:macro>
+  <xacro:include filename="util.xacro" />
   <!-- foot base link -->
   <link name="base_footprint">
