Commit message: every thing is ok

File: src/scene/urdf/camera.xacro (robot description, xacro)
@@ -4,5 +4,5 @@
     <visual>
       <geometry>
-        <cylinder radius="${camera_cylinder_radius}" length="${camera_cylinder_length}" />
+        <box size="${camera_box_radius} ${camera_box_radius} ${camera_box_radius}" />
       </geometry>
       <origin xyz="0.0 0.0 0.0" rpy="0.0 0.0 0.0" />
@@ -13,9 +13,9 @@
     <collision>
       <geometry>
-        <cylinder radius="${camera_cylinder_radius}" length="${camera_cylinder_length}" />
+        <box size="${camera_box_radius} ${camera_box_radius} ${camera_box_radius}" />
       </geometry>
       <origin xyz="0.0 0.0 0.0" rpy="0.0 0.0 0.0" />
     </collision>
-    <xacro:cylinder_inertial_matrix m="${camera_mass}" r="${camera_cylinder_radius}" h="${camera_cylinder_length}" />
+    <xacro:box_inertial_matrix m="${camera_mass}" l="${camera_box_radius}" w="${camera_box_radius}" h="${camera_box_radius}" />
   </link>
   <!-- joint -->
@@ -23,5 +23,5 @@
     <parent link="base_link" />
     <child link="camera" />
-    <origin xyz="0.0 ${base_box_size * 0.5 + camera_cylinder_length * 0.5} 0.0" rpy="${-PI * 0.5} 0.0 0.0" />
+    <origin xyz="${base_box_size * 0.5 + camera_box_radius * 0.5} 0.0 0.0" rpy="0.0 0.0 0.0" />
     <axis xyz="0.0 0.0 1.0" />
   </joint>

File: src/scene/urdf/imu.xacro (robot description, xacro)
@@ -23,5 +23,5 @@
     <parent link="base_link" />
     <child link="imu" />
-    <origin xyz="${base_box_size * 0.5 + imu_box_size * 0.5} 0.0 0.0" rpy="${PI} 0.0 0.0" />
+    <origin xyz="0.0 ${base_box_size * 0.5 + imu_box_size * 0.5} 0.0" rpy="0.0 0.0 0.0" />
     <axis xyz="0.0 0.0 1.0" />
   </joint>

File: src/scene/urdf/sensor-laser.xacro (robot description, xacro)
@@ -3,5 +3,5 @@
     <sensor type="ray" name="vodyne16">
       <pose>0 0 0 0 0 0</pose>
-      <visualize>true</visualize>
+      <visualize>false</visualize>
       <update_rate>5.5</update_rate>
       <ray>

File: src/scene/urdf/sim-robot.xacro (robot description, xacro)
@@ -5,6 +5,5 @@
   <xacro:property name="lidar_cylinder_radius" value="0.08" />
   <xacro:property name="lidar_cylinder_length" value="0.1" />
-  <xacro:property name="camera_cylinder_radius" value="0.05" />
-  <xacro:property name="camera_cylinder_length" value="0.05" />
+  <xacro:property name="camera_box_radius" value="0.1" />
   <xacro:property name="transparency" value="0.8" />
   <xacro:property name="PI" value="3.1415926535" />
