Commit message: update

File: src/scene/urdf/sensor-laser.xacro (robot description, xacro)
@@ -3,5 +3,5 @@
     <sensor type="ray" name="vodyne16">
       <pose>0 0 0 0 0 0</pose>
-      <visualize>false</visualize>
+      <visualize>true</visualize>
       <update_rate>5.5</update_rate>
       <ray>
@@ -33,5 +33,5 @@
       <plugin name="gazebo_rplidar" filename="libgazebo_ros_velodyne_laser.so">
         <topicName>/sim_lidar/scan</topicName>
-        <frameName>base_footprint</frameName>
+        <frameName>/lidar</frameName>
       </plugin>
     </sensor>

File: src/scene/urdf/sim-robot.xacro (robot description, xacro)
@@ -1,7 +1,7 @@
 <robot xmlns:xacro="http://www.ros.org/wiki/xacro" name="sim-robot">
   <xacro:property name="foot_box_size" value="0.001" />
-  <xacro:property name="base_box_size" value="0.3" />
+  <xacro:property name="base_box_size" value="0.2" />
   <xacro:property name="imu_box_size" value="0.1" />
-  <xacro:property name="lidar_cylinder_radius" value="0.08" />
+  <xacro:property name="lidar_cylinder_radius" value="0.05" />
   <xacro:property name="lidar_cylinder_length" value="0.1" />
   <xacro:property name="camera_box_radius" value="0.1" />
