Commit message: add wheels

File: src/scene/model/xacro/imu.xacro (robot description, xacro)
@@ -23,5 +23,5 @@
     <parent link="base_link" />
     <child link="imu" />
-    <origin xyz="0.0 ${base_box_size * 0.5 + imu_box_size * 0.5} 0.0" rpy="0.0 0.0 0.0" />
+    <origin xyz="-${base_box_size * 0.5 + imu_box_size * 0.5} 0.0 0.0" rpy="0.0 0.0 0.0" />
     <axis xyz="0.0 0.0 1.0" />
   </joint>

File: src/scene/model/xacro/sim-robot.xacro (robot description, xacro)
@@ -2,8 +2,11 @@
   <xacro:property name="foot_box_size" value="0.001" />
   <xacro:property name="base_box_size" value="0.2" />
-  <xacro:property name="imu_box_size" value="0.1" />
+  <xacro:property name="imu_box_size" value="0.06" />
   <xacro:property name="lidar_cylinder_radius" value="0.05" />
   <xacro:property name="lidar_cylinder_length" value="0.1" />
-  <xacro:property name="camera_box_radius" value="0.1" />
+  <xacro:property name="wheel_cylinder_radius" value="0.05" />
+  <xacro:property name="wheel_cylinder_length" value="0.03" />
+  <xacro:property name="ground_clearance" value="0.03" />
+  <xacro:property name="camera_box_radius" value="0.06" />
   <xacro:property name="transparency" value="0.8" />
   <xacro:property name="PI" value="3.1415926535" />
@@ -13,4 +16,6 @@
   <xacro:property name="imu_mass" value="1.0" />
   <xacro:property name="camera_mass" value="1.0" />
+  <xacro:property name="wheel_mass" value="1.0" />
+  <xacro:property name="support_wheel_mass" value="0.01" />
   <xacro:include filename="util.xacro" />
   <!-- foot base link -->
@@ -71,5 +76,5 @@
     <parent link="base_footprint" />
     <child link="base_link" />
-    <origin xyz="0.0 0.0 ${base_box_size * 0.5}" rpy="0.0 0.0 0.0" />
+    <origin xyz="0.0 0.0 ${base_box_size * 0.5 + ground_clearance}" rpy="0.0 0.0 0.0" />
     <axis xyz="0.0 0.0 1.0" />
   </joint>
@@ -80,3 +85,4 @@
   <xacro:include filename="sensor-imu.xacro" />
   <xacro:include filename="sensor-camera.xacro" />
+  <xacro:include filename="wheels.xacro" />
 </robot>
