Commit message: everything is fine

File: src/scene/model/xacro/motion.xacro (robot description, xacro)
@@ -33,5 +33,5 @@
       <wheelAcceleration>1.8</wheelAcceleration>
       <commandTopic>cmd_vel</commandTopic>
-      <odometryFrame>odom</odometryFrame>
+      <odometryFrame>map</odometryFrame>
       <odometryTopic>odom</odometryTopic>
       <robotBaseFrame>base_footprint</robotBaseFrame>

File: src/scene/model/xacro/sim-robot.xacro (robot description, xacro)
@@ -1,10 +1,10 @@
 <robot xmlns:xacro="http://www.ros.org/wiki/xacro" name="sim-robot">
   <xacro:property name="foot_box_size" value="0.001" />
-  <xacro:property name="base_box_size" value="0.2" />
+  <xacro:property name="base_box_size" value="0.3" />
   <xacro:property name="imu_box_size" value="0.06" />
   <xacro:property name="lidar_cylinder_radius" value="0.05" />
   <xacro:property name="lidar_cylinder_length" value="0.1" />
-  <xacro:property name="wheel_cylinder_radius" value="0.05" />
-  <xacro:property name="wheel_cylinder_length" value="0.03" />
+  <xacro:property name="wheel_cylinder_radius" value="0.08" />
+  <xacro:property name="wheel_cylinder_length" value="0.04" />
   <xacro:property name="ground_clearance" value="0.03" />
   <xacro:property name="camera_box_radius" value="0.06" />
@@ -16,6 +16,6 @@
   <xacro:property name="imu_mass" value="0.01" />
   <xacro:property name="camera_mass" value="0.01" />
-  <xacro:property name="wheel_mass" value="0.05" />
-  <xacro:property name="support_wheel_mass" value="0.03" />
+  <xacro:property name="wheel_mass" value="2.0" />
+  <xacro:property name="support_wheel_mass" value="2.0" />
   <xacro:include filename="util.xacro" />
   <!-- foot base link -->
