Commit message: everything is fine

File: src/scene/model/xacro/lidar.xacro (robot description, xacro)
@@ -1,3 +1,32 @@
 <robot xmlns:xacro="http://www.ros.org/wiki/xacro" name="lidar">
+  <!-- lidar -->
+  <link name="arm">
+    <visual>
+      <geometry>
+        <cylinder radius="${arm_cylinder_radius}" length="${arm_cylinder_length}" />
+      </geometry>
+      <origin xyz="0.0 0.0 0.0" rpy="0.0 0.0 0.0" />
+      <material name="black">
+        <color rgba="0.0 0.0 0.0 ${transparency}" />
+      </material>
+    </visual>
+    <collision>
+      <geometry>
+        <cylinder radius="${arm_cylinder_radius}" length="${arm_cylinder_length}" />
+      </geometry>
+      <origin xyz="0.0 0.0 0.0" rpy="0.0 0.0 0.0" />
+    </collision>
+    <xacro:cylinder_inertial_matrix m="${arm_mass}" r="${arm_cylinder_radius}" h="${arm_cylinder_length}" />
+  </link>
+  <!-- joint -->
+  <joint name="arm_to_base_link" type="fixed">
+    <parent link="base_link" />
+    <child link="arm" />
+    <origin xyz="0.0 0.0 ${base_box_size * 0.5 + arm_cylinder_length * 0.5}" rpy="0.0 0.0 0.0" />
+    <axis xyz="0.0 0.0 1.0" />
+  </joint>
+  <gazebo reference="arm">
+    <material>Gazebo/Black</material>
+  </gazebo>
   <!-- lidar -->
   <link name="lidar">
@@ -20,8 +49,8 @@
   </link>
   <!-- joint -->
-  <joint name="lidar_to_base_link" type="fixed">
-    <parent link="base_link" />
+  <joint name="lidar_to_arm" type="fixed">
+    <parent link="arm" />
     <child link="lidar" />
-    <origin xyz="0.0 0.0 ${base_box_size * 0.5 + lidar_cylinder_length * 0.5}" rpy="0.0 0.0 0.0" />
+    <origin xyz="0.0 0.0 ${arm_cylinder_length * 0.5 + lidar_cylinder_length * 0.5}" rpy="0.0 0.0 0.0" />
     <axis xyz="0.0 0.0 1.0" />
   </joint>

File: src/scene/model/xacro/motion.xacro (robot description, xacro)
@@ -18,8 +18,10 @@
     <plugin name="differential_drive_controller" filename="libgazebo_ros_diff_drive.so">
       <rosDebugLevel>Debug</rosDebugLevel>
-      <publishWheelTF>true</publishWheelTF>
+      <publishWheelTF>false</publishWheelTF>
       <robotNamespace>/</robotNamespace>
       <publishTf>1</publishTf>
-      <publishWheelJointState>true</publishWheelJointState>
+      <publishWheelJointState>false</publishWheelJointState>
+      <publishOdomTF>true</publishOdomTF>
+      <odometrySource>world</odometrySource>
       <alwaysOn>true</alwaysOn>
       <updateRate>100.0</updateRate>

File: src/scene/model/xacro/sensor-camera.xacro (robot description, xacro)
@@ -39,5 +39,5 @@
     <plugin name="camera_pose" filename="libgazebo_ros_p3d.so">
       <alwaysOn>true</alwaysOn>
-      <updateRate>30.0</updateRate>
+      <updateRate>50.0</updateRate>
       <bodyName>camera</bodyName>
       <topicName>camera_ground_truth</topicName>

File: src/scene/model/xacro/sensor-imu.xacro (robot description, xacro)
@@ -24,5 +24,5 @@
     <plugin name="imu_pose" filename="libgazebo_ros_p3d.so">
       <alwaysOn>true</alwaysOn>
-      <updateRate>400</updateRate>
+      <updateRate>50.0</updateRate>
       <bodyName>imu</bodyName>
       <topicName>imu_ground_truth</topicName>

File: src/scene/model/xacro/sensor-laser.xacro (robot description, xacro)
@@ -40,5 +40,5 @@
     <plugin name="lidar_pose" filename="libgazebo_ros_p3d.so">
       <alwaysOn>true</alwaysOn>
-      <updateRate>20.0</updateRate>
+      <updateRate>50.0</updateRate>
       <bodyName>lidar</bodyName>
       <topicName>lidar_ground_truth</topicName>

File: src/scene/model/xacro/sim-robot.xacro (robot description, xacro)
@@ -4,5 +4,7 @@
   <xacro:property name="imu_box_size" value="0.06" />
   <xacro:property name="lidar_cylinder_radius" value="0.05" />
-  <xacro:property name="lidar_cylinder_length" value="0.1" />
+  <xacro:property name="lidar_cylinder_length" value="0.05" />
+  <xacro:property name="arm_cylinder_radius" value="0.01" />
+  <xacro:property name="arm_cylinder_length" value="0.1" />
   <xacro:property name="wheel_cylinder_radius" value="0.08" />
   <xacro:property name="wheel_cylinder_length" value="0.04" />
@@ -14,4 +16,5 @@
   <xacro:property name="base_mass" value="0.5" />
   <xacro:property name="lidar_mass" value="0.02" />
+  <xacro:property name="arm_mass" value="0.01" />
   <xacro:property name="imu_mass" value="0.01" />
   <xacro:property name="camera_mass" value="0.01" />
