Commit message: add motions

File: src/scene/model/xacro/sim-robot.xacro (robot description, xacro)
@@ -12,10 +12,10 @@
   <xacro:property name="PI" value="3.1415926535" />
   <xacro:property name="foot_mass" value="0.001" />
-  <xacro:property name="base_mass" value="20.0" />
-  <xacro:property name="lidar_mass" value="5.0" />
-  <xacro:property name="imu_mass" value="1.0" />
-  <xacro:property name="camera_mass" value="1.0" />
-  <xacro:property name="wheel_mass" value="1.0" />
-  <xacro:property name="support_wheel_mass" value="0.01" />
+  <xacro:property name="base_mass" value="0.5" />
+  <xacro:property name="lidar_mass" value="0.02" />
+  <xacro:property name="imu_mass" value="0.01" />
+  <xacro:property name="camera_mass" value="0.01" />
+  <xacro:property name="wheel_mass" value="0.05" />
+  <xacro:property name="support_wheel_mass" value="0.03" />
   <xacro:include filename="util.xacro" />
   <!-- foot base link -->
@@ -29,10 +29,4 @@
       </material>
     </visual>
-    <collision>
-      <geometry>
-        <box size="${foot_box_size} ${foot_box_size} ${foot_box_size}" />
-      </geometry>
-      <origin xyz="0.0 0.0 0.0" rpy="0.0 0.0 0.0" />
-    </collision>
   </link>
   <gazebo reference="base_footprint">
@@ -86,3 +80,4 @@
   <xacro:include filename="sensor-camera.xacro" />
   <xacro:include filename="wheels.xacro" />
+  <xacro:include filename="motion.xacro" />
 </robot>

File: src/scene/model/xacro/wheels.xacro (robot description, xacro)
@@ -7,5 +7,5 @@
           <cylinder radius="${wheel_cylinder_radius}" length="${wheel_cylinder_length}" />
         </geometry>
-        <origin xyz="0.0 0.0 0.0" rpy="0.0 0.0 0.0" />
+        <origin xyz="0.0 0.0 0.0" rpy="${PI * 0.5} 0.0 0.0" />
         <material name="black">
           <color rgba="0.0 0.0 0.0 ${transparency}" />
@@ -16,5 +16,5 @@
           <cylinder radius="${wheel_cylinder_radius}" length="${wheel_cylinder_length}" />
         </geometry>
-        <origin xyz="0.0 0.0 0.0" rpy="0.0 0.0 0.0" />
+        <origin xyz="0.0 0.0 0.0" rpy="${PI * 0.5} 0.0 0.0" />
       </collision>
       <xacro:cylinder_inertial_matrix m="${wheel_mass}" r="${wheel_cylinder_radius}" h="${wheel_cylinder_length}" />
@@ -24,6 +24,6 @@
       <parent link="base_link" />
       <child link="${name}_wheel" />
-      <origin xyz="0.0 ${flag * (base_box_size * 0.5 + wheel_cylinder_length * 0.5)} -${base_box_size * 0.5 + ground_clearance - wheel_cylinder_radius}" rpy="${flag * PI * 0.5} 0.0 0.0" />
-      <axis xyz="0 0 1" />
+      <origin xyz="0.0 ${flag * base_box_size * 0.5} -${base_box_size * 0.5 + ground_clearance - wheel_cylinder_radius}"/>
+      <axis xyz="0 1 0" />
     </joint>
     <gazebo reference="${name}_wheel">
@@ -56,5 +56,5 @@
       <parent link="base_link" />
       <child link="${name}_support_wheel" />
-      <origin xyz="${flag * (base_box_size * 0.5 - ground_clearance * 0.5)} 0.0 -${base_box_size * 0.5 + ground_clearance * 0.5}" rpy="0.0 0.0 0.0" />
+      <origin xyz="${flag * (base_box_size * 0.5 - ground_clearance * 0.5)} 0.0 -${base_box_size * 0.5 + ground_clearance * 0.5}"/>
       <axis xyz="1 1 1" />
     </joint>

Commit message: add keyboard_teleop.launch

File: src/scene/model/xacro/sim-robot.xacro (robot description, xacro)
@@ -19,6 +19,6 @@
   <xacro:property name="imu_mass" value="0.01" />
   <xacro:property name="camera_mass" value="0.01" />
-  <xacro:property name="wheel_mass" value="2.0" />
-  <xacro:property name="support_wheel_mass" value="2.0" />
+  <xacro:property name="wheel_mass" value="0.3" />
+  <xacro:property name="support_wheel_mass" value="0.3" />
   <xacro:include filename="util.xacro" />
   <!-- foot base link -->
