Commit message: update

File: src/scene/model/xacro/camera.xacro (robot description, xacro)
@@ -7,6 +7,6 @@
       </geometry>
       <origin xyz="0.0 0.0 0.0" rpy="0.0 0.0 0.0" />
-      <material name="blue">
-        <color rgba="0.0 0.0 1.0 ${transparency}" />
+      <material name="green">
+        <color rgba="0.0 1.0 0.0 ${transparency}" />
       </material>
     </visual>

File: src/scene/model/xacro/imu.xacro (robot description, xacro)
@@ -7,6 +7,6 @@
       </geometry>
       <origin xyz="0.0 0.0 0.0" rpy="0.0 0.0 0.0" />
-      <material name="green">
-        <color rgba="0.0 1.0 0.0 ${transparency}" />
+      <material name="red">
+        <color rgba="1.0 0.0 0.0 ${transparency}" />
       </material>
     </visual>

File: src/scene/model/xacro/lidar.xacro (robot description, xacro)
@@ -36,6 +36,6 @@
       </geometry>
       <origin xyz="0.0 0.0 0.0" rpy="0.0 0.0 0.0" />
-      <material name="red">
-        <color rgba="1.0 0.0 0.0 ${transparency}" />
+      <material name="blue">
+        <color rgba="0.0 0.0 1.0 ${transparency}" />
       </material>
     </visual>

File: src/scene/model/xacro/sensor-imu.xacro (robot description, xacro)
@@ -24,5 +24,5 @@
     <plugin name="imu_pose" filename="libgazebo_ros_p3d.so">
       <alwaysOn>true</alwaysOn>
-      <updateRate>400.0</updateRate>
+      <updateRate>1000.0</updateRate>
       <bodyName>imu</bodyName>
       <topicName>imu_ground_truth</topicName>

File: src/scene/model/xacro/sensor-lidar.xacro (robot description, xacro)
@@ -14,6 +14,6 @@
           </horizontal>
           <vertical>
-            <samples>16</samples>
-            <resolution>2</resolution>
+            <samples>32</samples>
+            <resolution>1</resolution>
             <min_angle>-${15*PI/180.0}</min_angle>
             <max_angle> ${15*PI/180.0}</max_angle>
