Commit message: link robot to arm

File: src/arm_robot/model/robot/robot.xacro (robot description, xacro)
@@ -46,5 +46,5 @@
     <parent link="link4" />
     <child link="base_link" />
-    <origin xyz="${link4_length - base_box_size * 0.5} ${base_box_size} 0.0" rpy="0 0 0" />
+    <origin xyz="${link4_length - base_box_size * 0.5} ${base_box_size * 0.5 + link4_width * 0.5} 0.0" rpy="0 0 0" />
     <axis xyz="0 1 0" />
   </joint>
