Commit message: fine

File: src/arm_robot/model/robot/camera.xacro (robot description, xacro)
@@ -4,5 +4,5 @@
     <visual>
       <geometry>
-        <box size="${camera_box_radius} ${camera_box_radius} ${camera_box_radius}" />
+        <box size="${camera_box_size} ${camera_box_size} ${camera_box_size}" />
       </geometry>
       <origin xyz="0.0 0.0 0.0" rpy="0.0 0.0 0.0" />
@@ -13,9 +13,9 @@
     <collision>
       <geometry>
-        <box size="${camera_box_radius} ${camera_box_radius} ${camera_box_radius}" />
+        <box size="${camera_box_size} ${camera_box_size} ${camera_box_size}" />
       </geometry>
       <origin xyz="0.0 0.0 0.0" rpy="0.0 0.0 0.0" />
     </collision>
-    <xacro:box_inertial_matrix m="${camera_mass}" l="${camera_box_radius}" w="${camera_box_radius}" h="${camera_box_radius}" />
+    <xacro:box_inertial_matrix m="${camera_mass}" l="${camera_box_size}" w="${camera_box_size}" h="${camera_box_size}" />
   </link>
   <!-- joint -->
@@ -23,5 +23,5 @@
     <parent link="base_link" />
     <child link="camera" />
-    <origin xyz="${base_box_size * 0.5 + camera_box_radius * 0.5} 0.0 0.0" rpy="0.0 0.0 0.0" />
+    <origin xyz="${base_box_size * 0.5 + camera_box_size * 0.5} 0.0 0.0" rpy="0.0 0.0 0.0" />
     <axis xyz="0.0 0.0 1.0" />
   </joint>
