Commit message: fine

File: src/arm_robot/model/arm_robot.xacro (robot description, xacro)
@@ -1,3 +1,6 @@
 <robot xmlns:xacro="http://www.ros.org/wiki/xacro" name="robot">
+  <!-- ========================= -->
+  <!-- |    for arm params   | -->
+  <!-- ========================= -->
   <xacro:property name="link0_length" value="10.0" />
   <xacro:property name="link0_width" value="0.1" />
@@ -18,10 +21,29 @@
   <xacro:property name="platform_mass" value="100.0" />
   <xacro:property name="link_mass" value="0.001" />
+  <!-- ========================= -->
+  <!-- |    for robot params   | -->
+  <!-- ========================= -->
+  <xacro:property name="base_box_size" value="0.06" />
+  <xacro:property name="imu_box_size" value="0.04" />
+  <xacro:property name="lidar_cylinder_radius" value="0.03" />
+  <xacro:property name="lidar_cylinder_length" value="0.03" />
+  <xacro:property name="arm_cylinder_radius" value="0.005" />
+  <xacro:property name="arm_cylinder_length" value="0.06" />
+  <xacro:property name="wheel_cylinder_radius" value="0.08" />
+  <xacro:property name="wheel_cylinder_length" value="0.04" />
+  <xacro:property name="ground_clearance" value="0.03" />
+  <xacro:property name="camera_box_radius" value="0.04" />
+  <xacro:property name="transparency" value="0.8" />
+  <xacro:property name="PI" value="3.1415926535" />
+  <xacro:property name="foot_mass" value="0.001" />
+  <xacro:property name="base_mass" value="0.5" />
+  <xacro:property name="lidar_mass" value="0.02" />
+  <xacro:property name="arm_mass" value="0.01" />
+  <xacro:property name="imu_mass" value="0.01" />
+  <xacro:property name="camera_mass" value="0.01" />
+  <xacro:property name="wheel_mass" value="0.3" />
+  <xacro:property name="support_wheel_mass" value="0.3" />
   <xacro:include filename="$(find arm_robot)/model/util/util.xacro" />
   <xacro:include filename="$(find arm_robot)/model/arm/arm.xacro" />
-  <!--
-  <gazebo>
-    <plugin name="gazebo_ros_control" filename="libgazebo_ros_control.so"></plugin>
-  </gazebo> -->
   <xacro:include filename="$(find arm_robot)/model/robot/robot.xacro" />
   <xacro:gazebo-joint joint="link0_to_platform" transmission="hardware_interface/PositionJointInterface" />
@@ -43,3 +65,6 @@
   <xacro:gazebo-joint joint="base_to_link4" transmission="hardware_interface/VelocityJointInterface" />
   <xacro:gazebo-joint joint="base_to_link4" transmission="hardware_interface/EffortJointInterface" />
+  <gazebo>
+    <plugin name="gazebo_ros_control" filename="libgazebo_ros_control.so"></plugin>
+  </gazebo>
 </robot>

File: src/arm_robot/model/robot/robot.xacro (robot description, xacro)
@@ -1,24 +1,3 @@
 <robot xmlns:xacro="http://www.ros.org/wiki/xacro" name="sim-robot">
-  <xacro:property name="foot_box_size" value="0.001" />
-  <xacro:property name="base_box_size" value="0.3" />
-  <xacro:property name="imu_box_size" value="0.06" />
-  <xacro:property name="lidar_cylinder_radius" value="0.05" />
-  <xacro:property name="lidar_cylinder_length" value="0.05" />
-  <xacro:property name="arm_cylinder_radius" value="0.01" />
-  <xacro:property name="arm_cylinder_length" value="0.1" />
-  <xacro:property name="wheel_cylinder_radius" value="0.08" />
-  <xacro:property name="wheel_cylinder_length" value="0.04" />
-  <xacro:property name="ground_clearance" value="0.03" />
-  <xacro:property name="camera_box_radius" value="0.06" />
-  <xacro:property name="transparency" value="0.8" />
-  <xacro:property name="PI" value="3.1415926535" />
-  <xacro:property name="foot_mass" value="0.001" />
-  <xacro:property name="base_mass" value="0.5" />
-  <xacro:property name="lidar_mass" value="0.02" />
-  <xacro:property name="arm_mass" value="0.01" />
-  <xacro:property name="imu_mass" value="0.01" />
-  <xacro:property name="camera_mass" value="0.01" />
-  <xacro:property name="wheel_mass" value="0.3" />
-  <xacro:property name="support_wheel_mass" value="0.3" />
   <!-- base link -->
   <link name="base_link">

Commit message: fine

File: src/arm_robot/model/arm_robot.xacro (robot description, xacro)
@@ -33,5 +33,5 @@
   <xacro:property name="wheel_cylinder_length" value="0.04" />
   <xacro:property name="ground_clearance" value="0.03" />
-  <xacro:property name="camera_box_radius" value="0.04" />
+  <xacro:property name="camera_box_size" value="0.04" />
   <xacro:property name="transparency" value="0.8" />
   <xacro:property name="PI" value="3.1415926535" />

Commit message: fine

File: src/arm_robot/model/arm_robot.xacro (robot description, xacro)
@@ -6,17 +6,15 @@
   <!-- ========================= -->
   <xacro:property name="link0_length" value="10.0" />
-  <xacro:property name="link0_width" value="0.1" />
+  <xacro:property name="link0_width" value="0.06" />
   <xacro:property name="link1_length" value="0.3" />
-  <xacro:property name="link1_width" value="0.1" />
+  <xacro:property name="link1_width" value="0.06" />
   <xacro:property name="link2_length" value="3.0" />
-  <xacro:property name="link2_width" value="0.1" />
+  <xacro:property name="link2_width" value="0.06" />
   <xacro:property name="link3_length" value="0.1" />
-  <xacro:property name="link3_width" value="0.1" />
+  <xacro:property name="link3_width" value="0.06" />
   <xacro:property name="link4_length" value="0.2" />
-  <xacro:property name="link4_width" value="0.1" />
+  <xacro:property name="link4_width" value="0.06" />
   <xacro:property name="link5_length" value="0.1" />
-  <xacro:property name="link5_width" value="0.1" />
-  <xacro:property name="head_size" value="0.1" />
-  <xacro:property name="head_mass" value="0.001" />
+  <xacro:property name="link5_width" value="0.06" />
   <xacro:property name="platform_width" value="10.0" />
   <xacro:property name="platform_length" value="0.1" />

Commit message: fine

File: src/arm_robot/model/arm_robot.xacro (robot description, xacro)
@@ -35,10 +35,9 @@
   <xacro:property name="camera_box_size" value="0.04" />
   <xacro:property name="PI" value="3.1415926535" />
-  <xacro:property name="foot_mass" value="0.001" />
-  <xacro:property name="base_mass" value="0.5" />
-  <xacro:property name="lidar_mass" value="0.02" />
-  <xacro:property name="arm_mass" value="0.01" />
-  <xacro:property name="imu_mass" value="0.01" />
-  <xacro:property name="camera_mass" value="0.01" />
+  <xacro:property name="base_mass" value="0.001" />
+  <xacro:property name="lidar_mass" value="0.001" />
+  <xacro:property name="arm_mass" value="0.001" />
+  <xacro:property name="imu_mass" value="0.001" />
+  <xacro:property name="camera_mass" value="0.001" />
   <!-- ========================= -->
   <!-- | for link robot and arm| -->

Commit message: change mass

File: src/arm_robot/model/arm_robot.xacro (robot description, xacro)
@@ -35,9 +35,9 @@
   <xacro:property name="camera_box_size" value="0.04" />
   <xacro:property name="PI" value="3.1415926535" />
-  <xacro:property name="base_mass" value="0.0001" />
-  <xacro:property name="lidar_mass" value="0.0001" />
-  <xacro:property name="arm_mass" value="0.0001" />
-  <xacro:property name="imu_mass" value="0.0001" />
-  <xacro:property name="camera_mass" value="0.0001" />
+  <xacro:property name="base_mass" value="0.000" />
+  <xacro:property name="lidar_mass" value="0.000" />
+  <xacro:property name="arm_mass" value="0.000" />
+  <xacro:property name="imu_mass" value="0.000" />
+  <xacro:property name="camera_mass" value="0.000" />
   <!-- ========================= -->
   <!-- | for link robot and arm| -->

Commit message: change mass

File: src/arm_robot/model/arm_robot.xacro (robot description, xacro)
@@ -35,9 +35,9 @@
   <xacro:property name="camera_box_size" value="0.04" />
   <xacro:property name="PI" value="3.1415926535" />
-  <xacro:property name="base_mass" value="0.000" />
-  <xacro:property name="lidar_mass" value="0.000" />
-  <xacro:property name="arm_mass" value="0.000" />
-  <xacro:property name="imu_mass" value="0.000" />
-  <xacro:property name="camera_mass" value="0.000" />
+  <xacro:property name="base_mass" value="0.000001" />
+  <xacro:property name="lidar_mass" value="0.000001" />
+  <xacro:property name="arm_mass" value="0.000001" />
+  <xacro:property name="imu_mass" value="0.000001" />
+  <xacro:property name="camera_mass" value="0.000001" />
   <!-- ========================= -->
   <!-- | for link robot and arm| -->

Commit message: fine

File: src/arm_robot/model/arm_robot.xacro (robot description, xacro)
@@ -6,9 +6,9 @@
   <!-- ========================= -->
   <xacro:property name="link0_length" value="10.0" />
-  <xacro:property name="link0_width" value="0.06" />
+  <xacro:property name="link0_width" value="0.1" />
   <xacro:property name="link1_length" value="0.3" />
-  <xacro:property name="link1_width" value="0.06" />
+  <xacro:property name="link1_width" value="0.1" />
   <xacro:property name="link2_length" value="3.0" />
-  <xacro:property name="link2_width" value="0.06" />
+  <xacro:property name="link2_width" value="0.1" />
   <xacro:property name="link3_length" value="0.1" />
   <xacro:property name="link3_width" value="0.06" />

Commit message: update

File: src/arm_robot/model/arm_robot.xacro (robot description, xacro)
@@ -35,9 +35,9 @@
   <xacro:property name="camera_box_size" value="0.04" />
   <xacro:property name="PI" value="3.1415926535" />
-  <xacro:property name="base_mass" value="0.000001" />
-  <xacro:property name="lidar_mass" value="0.000001" />
-  <xacro:property name="arm_mass" value="0.000001" />
-  <xacro:property name="imu_mass" value="0.000001" />
-  <xacro:property name="camera_mass" value="0.000001" />
+  <xacro:property name="base_mass" value="1E-10" />
+  <xacro:property name="lidar_mass" value="1E-10" />
+  <xacro:property name="arm_mass" value="1E-10" />
+  <xacro:property name="imu_mass" value="1E-10" />
+  <xacro:property name="camera_mass" value="1E-10" />
   <!-- ========================= -->
   <!-- | for link robot and arm| -->

Commit message: update

File: src/arm_robot/model/arm_robot.xacro (robot description, xacro)
@@ -35,9 +35,9 @@
   <xacro:property name="camera_box_size" value="0.04" />
   <xacro:property name="PI" value="3.1415926535" />
-  <xacro:property name="base_mass" value="1E-10" />
-  <xacro:property name="lidar_mass" value="1E-10" />
-  <xacro:property name="arm_mass" value="1E-10" />
-  <xacro:property name="imu_mass" value="1E-10" />
-  <xacro:property name="camera_mass" value="1E-10" />
+  <xacro:property name="base_mass" value="0.001" />
+  <xacro:property name="lidar_mass" value="0.001" />
+  <xacro:property name="arm_mass" value="0.001" />
+  <xacro:property name="imu_mass" value="0.001" />
+  <xacro:property name="camera_mass" value="0.001" />
   <!-- ========================= -->
   <!-- | for link robot and arm| -->

Commit message: update

File: src/arm_robot/model/arm_robot.xacro (robot description, xacro)
@@ -29,5 +29,5 @@
   <xacro:property name="lidar_cylinder_length" value="0.03" />
   <xacro:property name="arm_cylinder_radius" value="0.005" />
-  <xacro:property name="arm_cylinder_length" value="0.06" />
+  <xacro:property name="arm_cylinder_length" value="0.04" />
   <xacro:property name="wheel_cylinder_radius" value="0.08" />
   <xacro:property name="wheel_cylinder_length" value="0.04" />

Commit message: update arm prams

File: src/arm_robot/model/arm_robot.xacro (robot description, xacro)
@@ -7,11 +7,11 @@
   <xacro:property name="link0_length" value="10.0" />
   <xacro:property name="link0_width" value="0.06" />
-  <xacro:property name="link1_length" value="0.3" />
+  <xacro:property name="link1_length" value="0.06" />
   <xacro:property name="link1_width" value="0.06" />
   <xacro:property name="link2_length" value="3.0" />
   <xacro:property name="link2_width" value="0.06" />
-  <xacro:property name="link3_length" value="0.1" />
+  <xacro:property name="link3_length" value="0.06" />
   <xacro:property name="link3_width" value="0.06" />
-  <xacro:property name="link4_length" value="0.2" />
+  <xacro:property name="link4_length" value="0.15" />
   <xacro:property name="link4_width" value="0.06" />
   <xacro:property name="link5_length" value="0.1" />
@@ -29,5 +29,5 @@
   <xacro:property name="lidar_cylinder_length" value="0.03" />
   <xacro:property name="arm_cylinder_radius" value="0.005" />
-  <xacro:property name="arm_cylinder_length" value="0.04" />
+  <xacro:property name="arm_cylinder_length" value="0.03" />
   <xacro:property name="wheel_cylinder_radius" value="0.08" />
   <xacro:property name="wheel_cylinder_length" value="0.04" />

Commit message: update arm prams

File: src/arm_robot/model/arm_robot.xacro (robot description, xacro)
@@ -9,5 +9,5 @@
   <xacro:property name="link1_length" value="0.06" />
   <xacro:property name="link1_width" value="0.06" />
-  <xacro:property name="link2_length" value="2.0" />
+  <xacro:property name="link2_length" value="3.0" />
   <xacro:property name="link2_width" value="0.06" />
   <xacro:property name="link3_length" value="0.06" />

Commit message: update arm prams

File: src/arm_robot/model/arm_robot.xacro (robot description, xacro)
@@ -11,5 +11,5 @@
   <xacro:property name="link2_length" value="3.0" />
   <xacro:property name="link2_width" value="0.06" />
-  <xacro:property name="link3_length" value="0.06" />
+  <xacro:property name="link3_length" value="0.1" />
   <xacro:property name="link3_width" value="0.06" />
   <xacro:property name="link4_length" value="0.15" />

Commit message: update arm prams

File: src/arm_robot/model/arm_robot.xacro (robot description, xacro)
@@ -7,5 +7,5 @@
   <xacro:property name="link0_length" value="10.0" />
   <xacro:property name="link0_width" value="0.06" />
-  <xacro:property name="link1_length" value="0.06" />
+  <xacro:property name="link1_length" value="0.2" />
   <xacro:property name="link1_width" value="0.06" />
   <xacro:property name="link2_length" value="3.0" />
