Commit message: add arm_robot

File: src/arm_robot/model/arm/arm.xacro (robot description, xacro)
@@ -47,60 +47,4 @@
     <material>Gazebo/Blue</material>
   </gazebo>
-  <link name="link0">
-    <visual>
-      <geometry>
-        <box size="${link0_length} ${link0_width} ${link0_width}" />
-      </geometry>
-      <material name="red">
-        <color rgba="1.0 0 0 0.5" />
-      </material>
-      <origin xyz="0.0 0.0 ${link0_width * 0.5}" rpy="0 0 0" />
-    </visual>
-    <collision>
-      <geometry>
-        <box size="${link0_length} ${link0_width} ${link0_width}" />
-      </geometry>
-      <origin xyz="0.0 0.0 ${link0_width * 0.5}" rpy="0 0 0" />
-    </collision>
-    <xacro:box_inertial_matrix m="${link_mass}" l="${link0_length}" w="${link0_width}" h="${link0_width}" />
-  </link>
-  <joint name="link0_to_base" type="prismatic">
-    <parent link="base" />
-    <child link="link0" />
-    <origin xyz="0.0 0.0 ${base_length}" rpy="0 0 0" />
-    <axis xyz="0 1 0" />
-    <limit lower="-${base_width * 0.5 - link0_width * 0.5}" upper="${base_width * 0.5 - link0_width * 0.5}" effort="10.0" velocity="1.0" />
-  </joint>
-  <gazebo reference="link0">
-    <material>Gazebo/Red</material>
-  </gazebo>
-  <link name="link1">
-    <visual>
-      <geometry>
-        <box size="${link1_width} ${link1_width} ${link1_length}" />
-      </geometry>
-      <material name="green">
-        <color rgba="0 1.0 0 0.5" />
-      </material>
-      <origin xyz="0.0 0.0 ${link1_length * 0.5}" rpy="0 0 0" />
-    </visual>
-    <collision>
-      <geometry>
-        <box size="${link1_width} ${link1_width} ${link1_length}" />
-      </geometry>
-      <origin xyz="0.0 0.0 ${link1_length * 0.5}" rpy="0 0 0" />
-    </collision>
-    <xacro:box_inertial_matrix m="${link_mass}" l="${link1_width}" w="${link1_width}" h="${link1_length}" />
-  </link>
-  <joint name="link1_to_link0" type="prismatic">
-    <parent link="link0" />
-    <child link="link1" />
-    <origin xyz="0.0 0.0 ${link0_width}" rpy="0 0 0" />
-    <axis xyz="1 0 0" />
-    <limit lower="-${link0_length * 0.5 - link1_width * 0.5}" upper="${link0_length * 0.5 - link1_width * 0.5}" effort="10.0" velocity="1.0" />
-  </joint>
-  <gazebo reference="link1">
-    <material>Gazebo/Green</material>
-  </gazebo>
   <link name="link2">
     <visual>
@@ -122,8 +66,8 @@
   </link>
   /moveit_tutorials/doc/pilz_industrial_motion_planner/pilz_industrial_motion_planner.html
-  <joint name="link2_to_link1" type="continuous">
-    <parent link="link1" />
+  <joint name="link2_to_base" type="continuous">
+    <parent link="base" />
     <child link="link2" />
-    <origin xyz="0.0 0.0 ${link1_length}" rpy="0 0 0" />
+    <origin xyz="0.0 0.0 ${base_length}" rpy="0 0 0" />
     <axis xyz="0 0 1" />
   </joint>

Commit message: ...

File: src/arm_robot/model/arm/arm.xacro (robot description, xacro)
@@ -47,4 +47,60 @@
     <material>Gazebo/Blue</material>
   </gazebo>
+  <link name="link0">
+    <visual>
+      <geometry>
+        <box size="${link0_length} ${link0_width} ${link0_width}" />
+      </geometry>
+      <material name="red">
+        <color rgba="1.0 0 0 0.5" />
+      </material>
+      <origin xyz="0.0 0.0 ${link0_width * 0.5}" rpy="0 0 0" />
+    </visual>
+    <collision>
+      <geometry>
+        <box size="${link0_length} ${link0_width} ${link0_width}" />
+      </geometry>
+      <origin xyz="0.0 0.0 ${link0_width * 0.5}" rpy="0 0 0" />
+    </collision>
+    <xacro:box_inertial_matrix m="${link_mass}" l="${link0_length}" w="${link0_width}" h="${link0_width}" />
+  </link>
+  <joint name="link0_to_base" type="prismatic">
+    <parent link="base" />
+    <child link="link0" />
+    <origin xyz="0.0 0.0 ${base_length}" rpy="0 0 0" />
+    <axis xyz="0 1 0" />
+    <limit lower="-${base_width * 0.5 - link0_width * 0.5}" upper="${base_width * 0.5 - link0_width * 0.5}" effort="10.0" velocity="1.0" />
+  </joint>
+  <gazebo reference="link0">
+    <material>Gazebo/Red</material>
+  </gazebo>
+  <link name="link1">
+    <visual>
+      <geometry>
+        <box size="${link1_width} ${link1_width} ${link1_length}" />
+      </geometry>
+      <material name="green">
+        <color rgba="0 1.0 0 0.5" />
+      </material>
+      <origin xyz="0.0 0.0 ${link1_length * 0.5}" rpy="0 0 0" />
+    </visual>
+    <collision>
+      <geometry>
+        <box size="${link1_width} ${link1_width} ${link1_length}" />
+      </geometry>
+      <origin xyz="0.0 0.0 ${link1_length * 0.5}" rpy="0 0 0" />
+    </collision>
+    <xacro:box_inertial_matrix m="${link_mass}" l="${link1_width}" w="${link1_width}" h="${link1_length}" />
+  </link>
+  <joint name="link1_to_link0" type="prismatic">
+    <parent link="link0" />
+    <child link="link1" />
+    <origin xyz="0.0 0.0 ${link0_width}" rpy="0 0 0" />
+    <axis xyz="1 0 0" />
+    <limit lower="-${link0_length * 0.5 - link1_width * 0.5}" upper="${link0_length * 0.5 - link1_width * 0.5}" effort="10.0" velocity="1.0" />
+  </joint>
+  <gazebo reference="link1">
+    <material>Gazebo/Green</material>
+  </gazebo>
   <link name="link2">
     <visual>
@@ -66,8 +122,8 @@
   </link>
   /moveit_tutorials/doc/pilz_industrial_motion_planner/pilz_industrial_motion_planner.html
-  <joint name="link2_to_base" type="continuous">
-    <parent link="base" />
+  <joint name="link2_to_link1" type="continuous">
+    <parent link="link1" />
     <child link="link2" />
-    <origin xyz="0.0 0.0 ${base_length}" rpy="0 0 0" />
+    <origin xyz="0.0 0.0 ${link1_length}" rpy="0 0 0" />
     <axis xyz="0 0 1" />
   </joint>

Commit message: ...

File: src/arm_robot/model/arm/arm.xacro (robot description, xacro)
@@ -14,35 +14,35 @@
   <xacro:property name="head_size" value="0.1" />
   <xacro:property name="head_mass" value="0.001" />
-  <xacro:property name="base_width" value="10.0" />
-  <xacro:property name="base_length" value="0.1" />
-  <xacro:property name="base_mass" value="100.0" />
+  <xacro:property name="platform_width" value="10.0" />
+  <xacro:property name="platform_length" value="0.1" />
+  <xacro:property name="platform_mass" value="100.0" />
   <xacro:property name="link_mass" value="0.001" />
   <xacro:include filename="$(find arm_robot)/model/util/util.xacro" />
-  <link name="base_footprint"></link>
-  <link name="base">
-    <visual>
-      <geometry>
-        <box size="${base_width} ${base_width} ${base_length}" />
+  <link name="platform_footprint"></link>
+  <link name="platform">
+    <visual>
+      <geometry>
+        <box size="${platform_width} ${platform_width} ${platform_length}" />
       </geometry>
       <material name="blue">
         <color rgba="0 0 1.0 0.5" />
       </material>
-      <origin xyz="0.0 0.0 ${base_length * 0.5}" rpy="0 0 0" />
-    </visual>
-    <collision>
-      <geometry>
-        <box size="${base_width} ${base_width} ${base_length}" />
-      </geometry>
-      <origin xyz="0.0 0.0 ${base_length * 0.5}" rpy="0 0 0" />
-    </collision>
-    <xacro:box_inertial_matrix m="${base_mass}" l="${link0_length}" w="${base_width}" h="${base_length}" />
-  </link>
-  <joint name="base_to_footprint" type="fixed">
-    <parent link="base_footprint" />
-    <child link="base" />
+      <origin xyz="0.0 0.0 ${platform_length * 0.5}" rpy="0 0 0" />
+    </visual>
+    <collision>
+      <geometry>
+        <box size="${platform_width} ${platform_width} ${platform_length}" />
+      </geometry>
+      <origin xyz="0.0 0.0 ${platform_length * 0.5}" rpy="0 0 0" />
+    </collision>
+    <xacro:box_inertial_matrix m="${platform_mass}" l="${link0_length}" w="${platform_width}" h="${platform_length}" />
+  </link>
+  <joint name="platform_to_footprint" type="fixed">
+    <parent link="platform_footprint" />
+    <child link="platform" />
     <origin xyz="0.0 0.0 0.0" rpy="0 0 0" />
     <axis xyz="0 1 0" />
   </joint>
-  <gazebo reference="base">
+  <gazebo reference="platform">
     <material>Gazebo/Blue</material>
   </gazebo>
@@ -65,10 +65,10 @@
     <xacro:box_inertial_matrix m="${link_mass}" l="${link0_length}" w="${link0_width}" h="${link0_width}" />
   </link>
-  <joint name="link0_to_base" type="prismatic">
-    <parent link="base" />
+  <joint name="link0_to_platform" type="prismatic">
+    <parent link="platform" />
     <child link="link0" />
-    <origin xyz="0.0 0.0 ${base_length}" rpy="0 0 0" />
+    <origin xyz="0.0 0.0 ${platform_length}" rpy="0 0 0" />
     <axis xyz="0 1 0" />
-    <limit lower="-${base_width * 0.5 - link0_width * 0.5}" upper="${base_width * 0.5 - link0_width * 0.5}" effort="10.0" velocity="1.0" />
+    <limit lower="-${platform_width * 0.5 - link0_width * 0.5}" upper="${platform_width * 0.5 - link0_width * 0.5}" effort="10.0" velocity="1.0" />
   </joint>
   <gazebo reference="link0">
@@ -209,7 +209,7 @@
     <material>Gazebo/Yellow</material>
   </gazebo>
-  <xacro:gazebo-joint joint="link0_to_base" transmission="hardware_interface/PositionJointInterface" />
-  <xacro:gazebo-joint joint="link0_to_base" transmission="hardware_interface/VelocityJointInterface" />
-  <xacro:gazebo-joint joint="link0_to_base" transmission="hardware_interface/EffortJointInterface" />
+  <xacro:gazebo-joint joint="link0_to_platform" transmission="hardware_interface/PositionJointInterface" />
+  <xacro:gazebo-joint joint="link0_to_platform" transmission="hardware_interface/VelocityJointInterface" />
+  <xacro:gazebo-joint joint="link0_to_platform" transmission="hardware_interface/EffortJointInterface" />
   <xacro:gazebo-joint joint="link1_to_link0" transmission="hardware_interface/PositionJointInterface" />
   <xacro:gazebo-joint joint="link1_to_link0" transmission="hardware_interface/VelocityJointInterface" />

Commit message: rviz config file

File: src/arm_robot/model/arm/arm.xacro (robot description, xacro)
@@ -1,22 +1,3 @@
 <robot xmlns:xacro="http://www.ros.org/wiki/xacro" name="robot">
-  <xacro:property name="link0_length" value="10.0" />
-  <xacro:property name="link0_width" value="0.1" />
-  <xacro:property name="link1_length" value="0.3" />
-  <xacro:property name="link1_width" value="0.1" />
-  <xacro:property name="link2_length" value="3.0" />
-  <xacro:property name="link2_width" value="0.1" />
-  <xacro:property name="link3_length" value="0.1" />
-  <xacro:property name="link3_width" value="0.1" />
-  <xacro:property name="link4_length" value="0.2" />
-  <xacro:property name="link4_width" value="0.1" />
-  <xacro:property name="link5_length" value="0.1" />
-  <xacro:property name="link5_width" value="0.1" />
-  <xacro:property name="head_size" value="0.1" />
-  <xacro:property name="head_mass" value="0.001" />
-  <xacro:property name="platform_width" value="10.0" />
-  <xacro:property name="platform_length" value="0.1" />
-  <xacro:property name="platform_mass" value="100.0" />
-  <xacro:property name="link_mass" value="0.001" />
-  <xacro:include filename="$(find arm_robot)/model/util/util.xacro" />
   <link name="platform_footprint"></link>
   <link name="platform">

File: src/arm_robot/model/arm_robot.xacro (robot description, xacro)
@@ -1,3 +1,22 @@
 <robot xmlns:xacro="http://www.ros.org/wiki/xacro" name="robot">
-  <xacro:include filename="$(find arm_robot)/model/arm/arm.xacro"/>
+  <xacro:property name="link0_length" value="10.0" />
+  <xacro:property name="link0_width" value="0.1" />
+  <xacro:property name="link1_length" value="0.3" />
+  <xacro:property name="link1_width" value="0.1" />
+  <xacro:property name="link2_length" value="3.0" />
+  <xacro:property name="link2_width" value="0.1" />
+  <xacro:property name="link3_length" value="0.1" />
+  <xacro:property name="link3_width" value="0.1" />
+  <xacro:property name="link4_length" value="0.2" />
+  <xacro:property name="link4_width" value="0.1" />
+  <xacro:property name="link5_length" value="0.1" />
+  <xacro:property name="link5_width" value="0.1" />
+  <xacro:property name="head_size" value="0.1" />
+  <xacro:property name="head_mass" value="0.001" />
+  <xacro:property name="platform_width" value="10.0" />
+  <xacro:property name="platform_length" value="0.1" />
+  <xacro:property name="platform_mass" value="100.0" />
+  <xacro:property name="link_mass" value="0.001" />
+  <xacro:include filename="$(find arm_robot)/model/util/util.xacro" />
+  <xacro:include filename="$(find arm_robot)/model/arm/arm.xacro" />
 </robot>

Commit message: link robot to arm

File: src/arm_robot/model/arm/arm.xacro (robot description, xacro)
@@ -163,48 +163,3 @@
     <material>Gazebo/Red</material>
   </gazebo>
-  <link name="link5">
-    <visual>
-      <geometry>
-        <box size="${link5_width} ${link5_length} ${link5_width}" />
-      </geometry>
-      <material name="yellow">
-        <color rgba="1.0 1.0 0 0.5" />
-      </material>
-      <origin xyz="0.0 0.0 0.0" rpy="0 0 0" />
-    </visual>
-    <collision>
-      <geometry>
-        <box size="${link5_width} ${link5_length} ${link5_width}" />
-      </geometry>
-      <origin xyz="0.0 0.0 0.0" rpy="0 0 0" />
-    </collision>
-    <xacro:box_inertial_matrix m="${link_mass}" l="${link5_width}" w="${link5_length}" h="${link5_width}" />
-  </link>
-  <joint name="link5_to_link4" type="continuous">
-    <parent link="link4" />
-    <child link="link5" />
-    <origin xyz="${link4_length - link5_width * 0.5} ${link5_length} 0.0" rpy="0 0 0" />
-    <axis xyz="0 1 0" />
-  </joint>
-  <gazebo reference="link5">
-    <material>Gazebo/Yellow</material>
-  </gazebo>
-  <xacro:gazebo-joint joint="link0_to_platform" transmission="hardware_interface/PositionJointInterface" />
-  <xacro:gazebo-joint joint="link0_to_platform" transmission="hardware_interface/VelocityJointInterface" />
-  <xacro:gazebo-joint joint="link0_to_platform" transmission="hardware_interface/EffortJointInterface" />
-  <xacro:gazebo-joint joint="link1_to_link0" transmission="hardware_interface/PositionJointInterface" />
-  <xacro:gazebo-joint joint="link1_to_link0" transmission="hardware_interface/VelocityJointInterface" />
-  <xacro:gazebo-joint joint="link1_to_link0" transmission="hardware_interface/EffortJointInterface" />
-  <xacro:gazebo-joint joint="link2_to_link1" transmission="hardware_interface/PositionJointInterface" />
-  <xacro:gazebo-joint joint="link2_to_link1" transmission="hardware_interface/VelocityJointInterface" />
-  <xacro:gazebo-joint joint="link2_to_link1" transmission="hardware_interface/EffortJointInterface" />
-  <xacro:gazebo-joint joint="link3_to_link2" transmission="hardware_interface/PositionJointInterface" />
-  <xacro:gazebo-joint joint="link3_to_link2" transmission="hardware_interface/VelocityJointInterface" />
-  <xacro:gazebo-joint joint="link3_to_link2" transmission="hardware_interface/EffortJointInterface" />
-  <xacro:gazebo-joint joint="link4_to_link3" transmission="hardware_interface/PositionJointInterface" />
-  <xacro:gazebo-joint joint="link4_to_link3" transmission="hardware_interface/VelocityJointInterface" />
-  <xacro:gazebo-joint joint="link4_to_link3" transmission="hardware_interface/EffortJointInterface" />
-  <xacro:gazebo-joint joint="link5_to_link4" transmission="hardware_interface/PositionJointInterface" />
-  <xacro:gazebo-joint joint="link5_to_link4" transmission="hardware_interface/VelocityJointInterface" />
-  <xacro:gazebo-joint joint="link5_to_link4" transmission="hardware_interface/EffortJointInterface" />
 </robot>

File: src/arm_robot/model/arm_robot.xacro (robot description, xacro)
@@ -1,4 +1,3 @@
 <robot xmlns:xacro="http://www.ros.org/wiki/xacro" name="robot">
-<!--
   <xacro:property name="link0_length" value="10.0" />
   <xacro:property name="link0_width" value="0.1" />
@@ -21,7 +20,26 @@
   <xacro:include filename="$(find arm_robot)/model/util/util.xacro" />
   <xacro:include filename="$(find arm_robot)/model/arm/arm.xacro" />
+  <!--
   <gazebo>
     <plugin name="gazebo_ros_control" filename="libgazebo_ros_control.so"></plugin>
   </gazebo> -->
   <xacro:include filename="$(find arm_robot)/model/robot/robot.xacro" />
+  <xacro:gazebo-joint joint="link0_to_platform" transmission="hardware_interface/PositionJointInterface" />
+  <xacro:gazebo-joint joint="link0_to_platform" transmission="hardware_interface/VelocityJointInterface" />
+  <xacro:gazebo-joint joint="link0_to_platform" transmission="hardware_interface/EffortJointInterface" />
+  <xacro:gazebo-joint joint="link1_to_link0" transmission="hardware_interface/PositionJointInterface" />
+  <xacro:gazebo-joint joint="link1_to_link0" transmission="hardware_interface/VelocityJointInterface" />
+  <xacro:gazebo-joint joint="link1_to_link0" transmission="hardware_interface/EffortJointInterface" />
+  <xacro:gazebo-joint joint="link2_to_link1" transmission="hardware_interface/PositionJointInterface" />
+  <xacro:gazebo-joint joint="link2_to_link1" transmission="hardware_interface/VelocityJointInterface" />
+  <xacro:gazebo-joint joint="link2_to_link1" transmission="hardware_interface/EffortJointInterface" />
+  <xacro:gazebo-joint joint="link3_to_link2" transmission="hardware_interface/PositionJointInterface" />
+  <xacro:gazebo-joint joint="link3_to_link2" transmission="hardware_interface/VelocityJointInterface" />
+  <xacro:gazebo-joint joint="link3_to_link2" transmission="hardware_interface/EffortJointInterface" />
+  <xacro:gazebo-joint joint="link4_to_link3" transmission="hardware_interface/PositionJointInterface" />
+  <xacro:gazebo-joint joint="link4_to_link3" transmission="hardware_interface/VelocityJointInterface" />
+  <xacro:gazebo-joint joint="link4_to_link3" transmission="hardware_interface/EffortJointInterface" />
+  <xacro:gazebo-joint joint="base_to_link4" transmission="hardware_interface/PositionJointInterface" />
+  <xacro:gazebo-joint joint="base_to_link4" transmission="hardware_interface/VelocityJointInterface" />
+  <xacro:gazebo-joint joint="base_to_link4" transmission="hardware_interface/EffortJointInterface" />
 </robot>

File: src/arm_robot/model/robot/robot.xacro (robot description, xacro)
@@ -21,31 +21,4 @@
   <xacro:property name="wheel_mass" value="0.3" />
   <xacro:property name="support_wheel_mass" value="0.3" />
-  <xacro:include filename="util.xacro" />
-  <!-- foot base link -->
-  <link name="base_footprint">
-    <visual>
-      <geometry>
-        <box size="${foot_box_size} ${foot_box_size} ${foot_box_size}" />
-      </geometry>
-      <material name="black">
-        <color rgba="0.0 0.0 0.0 ${transparency}" />
-      </material>
-    </visual>
-  </link>
-  <gazebo reference="base_footprint">
-    <material>Gazebo/Black</material>
-  </gazebo>
-  <gazebo>
-    <plugin name="base_footprint_pose" filename="libgazebo_ros_p3d.so">
-      <alwaysOn>true</alwaysOn>
-      <updateRate>50.0</updateRate>
-      <bodyName>base_footprint</bodyName>
-      <topicName>base_footprint_ground_truth</topicName>
-      <gaussianNoise>0.0</gaussianNoise>
-      <frameName>map</frameName>
-      <xyzOffsets>0 0 0</xyzOffsets>
-      <rpyOffsets>0 0 0</rpyOffsets>
-    </plugin>
-  </gazebo>
   <!-- base link -->
   <link name="base_link">
@@ -70,9 +43,9 @@
   </gazebo>
   <!-- joint -->
-  <joint name="base_to_foot" type="fixed">
-    <parent link="base_footprint" />
+  <joint name="base_to_link4" type="continuous">
+    <parent link="link4" />
     <child link="base_link" />
-    <origin xyz="0.0 0.0 ${base_box_size * 0.5 + ground_clearance}" rpy="0.0 0.0 0.0" />
-    <axis xyz="0.0 0.0 1.0" />
+    <origin xyz="${link4_length - base_box_size * 0.5} ${base_box_size} 0.0" rpy="0 0 0" />
+    <axis xyz="0 1 0" />
   </joint>
   <xacro:include filename="lidar.xacro" />

Commit message: fine

File: src/arm_robot/model/arm/arm.xacro (robot description, xacro)
@@ -7,5 +7,5 @@
       </geometry>
       <material name="blue">
-        <color rgba="0 0 1.0 0.5" />
+        <color rgba="0 0 1.0 ${transparency}" />
       </material>
       <origin xyz="0.0 0.0 ${platform_length * 0.5}" rpy="0 0 0" />
@@ -34,5 +34,5 @@
       </geometry>
       <material name="red">
-        <color rgba="1.0 0 0 0.5" />
+        <color rgba="1.0 0 0 ${transparency}" />
       </material>
       <origin xyz="0.0 0.0 ${link0_width * 0.5}" rpy="0 0 0" />
@@ -62,5 +62,5 @@
       </geometry>
       <material name="green">
-        <color rgba="0 1.0 0 0.5" />
+        <color rgba="0 1.0 0 ${transparency}" />
       </material>
       <origin xyz="0.0 0.0 ${link1_length * 0.5}" rpy="0 0 0" />
@@ -90,5 +90,5 @@
       </geometry>
       <material name="blue">
-        <color rgba="0 0 1.0 0.5" />
+        <color rgba="0 0 1.0 ${transparency}" />
       </material>
       <origin xyz="0.0 0.0 ${link2_length * 0.5}" rpy="0 0 0" />

File: src/arm_robot/model/arm_robot.xacro (robot description, xacro)
@@ -1,3 +1,5 @@
 <robot xmlns:xacro="http://www.ros.org/wiki/xacro" name="robot">
+  <xacro:property name="transparency" value="0.8" />
+  <xacro:include filename="$(find arm_robot)/model/util/util.xacro" />
   <!-- ========================= -->
   <!-- |    for arm params   | -->
@@ -34,5 +36,4 @@
   <xacro:property name="ground_clearance" value="0.03" />
   <xacro:property name="camera_box_size" value="0.04" />
-  <xacro:property name="transparency" value="0.8" />
   <xacro:property name="PI" value="3.1415926535" />
   <xacro:property name="foot_mass" value="0.001" />
@@ -42,7 +43,7 @@
   <xacro:property name="imu_mass" value="0.01" />
   <xacro:property name="camera_mass" value="0.01" />
-  <xacro:property name="wheel_mass" value="0.3" />
-  <xacro:property name="support_wheel_mass" value="0.3" />
-  <xacro:include filename="$(find arm_robot)/model/util/util.xacro" />
+  <!-- ========================= -->
+  <!-- | for link robot and arm| -->
+  <!-- ========================= -->
   <xacro:include filename="$(find arm_robot)/model/arm/arm.xacro" />
   <xacro:include filename="$(find arm_robot)/model/robot/robot.xacro" />

Commit message: fine

File: src/arm_robot/model/arm/arm.xacro (robot description, xacro)
@@ -89,6 +89,6 @@
         <box size="${link2_width} ${link2_width} ${link2_length}" />
       </geometry>
-      <material name="blue">
-        <color rgba="0 0 1.0 ${transparency}" />
+      <material name="red">
+        <color rgba="1.0 0 0 ${transparency}" />
       </material>
       <origin xyz="0.0 0.0 ${link2_length * 0.5}" rpy="0 0 0" />
@@ -102,5 +102,4 @@
     <xacro:box_inertial_matrix m="${link_mass}" l="${link2_width}" w="${link2_width}" h="${link2_length}" />
   </link>
-  /moveit_tutorials/doc/pilz_industrial_motion_planner/pilz_industrial_motion_planner.html
   <joint name="link2_to_link1" type="continuous">
     <parent link="link1" />
@@ -110,5 +109,5 @@
   </joint>
   <gazebo reference="link2">
-    <material>Gazebo/Blue</material>
+    <material>Gazebo/Red</material>
   </gazebo>
   <link name="link3">
