Commit message: change mass

File: src/arm_robot/model/arm/arm.xacro (robot description, xacro)
@@ -52,4 +52,5 @@
     <axis xyz="0 1 0" />
     <limit lower="-${platform_width * 0.5 - link0_width * 0.5}" upper="${platform_width * 0.5 - link0_width * 0.5}" effort="10.0" velocity="1.0" />
+    <dynamics damping="0.7" friction="0.0" />
   </joint>
   <gazebo reference="link0">
@@ -80,4 +81,5 @@
     <axis xyz="1 0 0" />
     <limit lower="-${link0_length * 0.5 - link1_width * 0.5}" upper="${link0_length * 0.5 - link1_width * 0.5}" effort="10.0" velocity="1.0" />
+    <dynamics damping="0.7" friction="0.0" />
   </joint>
   <gazebo reference="link1">
@@ -107,4 +109,5 @@
     <origin xyz="0.0 0.0 ${link1_length}" rpy="0 0 0" />
     <axis xyz="0 0 1" />
+    <dynamics damping="0.7" friction="0.0" />
   </joint>
   <gazebo reference="link2">
@@ -133,4 +136,5 @@
     <axis xyz="0 0 1" />
     <limit lower="-${link2_length * 0.5 - link3_width * 0.5}" upper="${link2_length * 0.5 - link3_width * 0.5}" effort="10.0" velocity="1.0" />
+    <dynamics damping="0.7" friction="0.0" />
   </joint>
   <gazebo reference="link3">
@@ -158,4 +162,5 @@
     <origin xyz="${link3_length} 0.0 0.0" rpy="0 0 0" />
     <axis xyz="1 0 0" />
+    <dynamics damping="0.7" friction="0.0" />
   </joint>
   <gazebo reference="link4">

File: src/arm_robot/model/arm_robot.xacro (robot description, xacro)
@@ -20,5 +20,5 @@
   <xacro:property name="platform_length" value="0.1" />
   <xacro:property name="platform_mass" value="100.0" />
-  <xacro:property name="link_mass" value="0.001" />
+  <xacro:property name="link_mass" value="0.1" />
   <!-- ========================= -->
   <!-- |    for robot params   | -->
@@ -35,9 +35,9 @@
   <xacro:property name="camera_box_size" value="0.04" />
   <xacro:property name="PI" value="3.1415926535" />
-  <xacro:property name="base_mass" value="0.001" />
-  <xacro:property name="lidar_mass" value="0.001" />
-  <xacro:property name="arm_mass" value="0.001" />
-  <xacro:property name="imu_mass" value="0.001" />
-  <xacro:property name="camera_mass" value="0.001" />
+  <xacro:property name="base_mass" value="0.0001" />
+  <xacro:property name="lidar_mass" value="0.0001" />
+  <xacro:property name="arm_mass" value="0.0001" />
+  <xacro:property name="imu_mass" value="0.0001" />
+  <xacro:property name="camera_mass" value="0.0001" />
   <!-- ========================= -->
   <!-- | for link robot and arm| -->

Commit message: fine

File: src/arm_robot/model/arm/arm.xacro (robot description, xacro)
@@ -52,5 +52,5 @@
     <axis xyz="0 1 0" />
     <limit lower="-${platform_width * 0.5 - link0_width * 0.5}" upper="${platform_width * 0.5 - link0_width * 0.5}" effort="10.0" velocity="1.0" />
-    <dynamics damping="0.7" friction="0.0" />
+    <dynamics D="1" K="7000" damping="0.003" friction="0.0" mu_coulomb="0" mu_viscous="16" />
   </joint>
   <gazebo reference="link0">
@@ -81,5 +81,5 @@
     <axis xyz="1 0 0" />
     <limit lower="-${link0_length * 0.5 - link1_width * 0.5}" upper="${link0_length * 0.5 - link1_width * 0.5}" effort="10.0" velocity="1.0" />
-    <dynamics damping="0.7" friction="0.0" />
+    <dynamics D="1" K="7000" damping="0.003" friction="0.0" mu_coulomb="0" mu_viscous="16" />
   </joint>
   <gazebo reference="link1">
@@ -109,5 +109,5 @@
     <origin xyz="0.0 0.0 ${link1_length}" rpy="0 0 0" />
     <axis xyz="0 0 1" />
-    <dynamics damping="0.7" friction="0.0" />
+    <dynamics D="1" K="7000" damping="0.003" friction="0.0" mu_coulomb="0" mu_viscous="16" />
   </joint>
   <gazebo reference="link2">
@@ -136,5 +136,5 @@
     <axis xyz="0 0 1" />
     <limit lower="-${link2_length * 0.5 - link3_width * 0.5}" upper="${link2_length * 0.5 - link3_width * 0.5}" effort="10.0" velocity="1.0" />
-    <dynamics damping="0.7" friction="0.0" />
+    <dynamics D="1" K="7000" damping="0.003" friction="0.0" mu_coulomb="0" mu_viscous="16" />
   </joint>
   <gazebo reference="link3">
@@ -163,4 +163,5 @@
     <axis xyz="1 0 0" />
     <dynamics damping="0.7" friction="0.0" />
+    <dynamics D="1" K="7000" damping="0.003" friction="0.0" mu_coulomb="0" mu_viscous="16" />
   </joint>
   <gazebo reference="link4">

Commit message: update

File: src/arm_robot/model/arm/arm.xacro (robot description, xacro)
@@ -9,5 +9,4 @@
         <color rgba="0 0 1.0 ${transparency}" />
       </material>
-      <origin xyz="0.0 0.0 ${platform_length * 0.5}" rpy="0 0 0" />
     </visual>
     <collision>
@@ -15,12 +14,11 @@
         <box size="${platform_width} ${platform_width} ${platform_length}" />
       </geometry>
-      <origin xyz="0.0 0.0 ${platform_length * 0.5}" rpy="0 0 0" />
     </collision>
-    <xacro:box_inertial_matrix m="${platform_mass}" l="${link0_length}" w="${platform_width}" h="${platform_length}" />
+    <xacro:box_inertial_matrix m="${platform_mass}" l="${platform_width}" w="${platform_width}" h="${platform_length}" />
   </link>
   <joint name="platform_to_footprint" type="fixed">
     <parent link="platform_footprint" />
     <child link="platform" />
-    <origin xyz="0.0 0.0 0.0" rpy="0 0 0" />
+    <origin xyz="0.0 0.0 ${0.5 * platform_length}" rpy="0 0 0" />
     <axis xyz="0 1 0" />
   </joint>
@@ -36,5 +34,4 @@
         <color rgba="1.0 0 0 ${transparency}" />
       </material>
-      <origin xyz="0.0 0.0 ${link0_width * 0.5}" rpy="0 0 0" />
     </visual>
     <collision>
@@ -42,5 +39,4 @@
         <box size="${link0_length} ${link0_width} ${link0_width}" />
       </geometry>
-      <origin xyz="0.0 0.0 ${link0_width * 0.5}" rpy="0 0 0" />
     </collision>
     <xacro:box_inertial_matrix m="${link_mass}" l="${link0_length}" w="${link0_width}" h="${link0_width}" />
@@ -49,5 +45,5 @@
     <parent link="platform" />
     <child link="link0" />
-    <origin xyz="0.0 0.0 ${platform_length}" rpy="0 0 0" />
+    <origin xyz="0.0 0.0 ${platform_length * 0.5 + link0_width * 0.5}" rpy="0 0 0" />
     <axis xyz="0 1 0" />
     <limit lower="-${platform_width * 0.5 - link0_width * 0.5}" upper="${platform_width * 0.5 - link0_width * 0.5}" effort="10.0" velocity="1.0" />
@@ -65,5 +61,4 @@
         <color rgba="0 1.0 0 ${transparency}" />
       </material>
-      <origin xyz="0.0 0.0 ${link1_length * 0.5}" rpy="0 0 0" />
     </visual>
     <collision>
@@ -71,5 +66,4 @@
         <box size="${link1_width} ${link1_width} ${link1_length}" />
       </geometry>
-      <origin xyz="0.0 0.0 ${link1_length * 0.5}" rpy="0 0 0" />
     </collision>
     <xacro:box_inertial_matrix m="${link_mass}" l="${link1_width}" w="${link1_width}" h="${link1_length}" />
@@ -78,5 +72,5 @@
     <parent link="link0" />
     <child link="link1" />
-    <origin xyz="0.0 0.0 ${link0_width}" rpy="0 0 0" />
+    <origin xyz="0.0 0.0 ${link0_width * 0.5 + link1_length * 0.5}" rpy="0 0 0" />
     <axis xyz="1 0 0" />
     <limit lower="-${link0_length * 0.5 - link1_width * 0.5}" upper="${link0_length * 0.5 - link1_width * 0.5}" effort="10.0" velocity="1.0" />
@@ -94,5 +88,4 @@
         <color rgba="1.0 0 0 ${transparency}" />
       </material>
-      <origin xyz="0.0 0.0 ${link2_length * 0.5}" rpy="0 0 0" />
     </visual>
     <collision>
@@ -100,5 +93,4 @@
         <box size="${link2_width} ${link2_width} ${link2_length}" />
       </geometry>
-      <origin xyz="0.0 0.0 ${link2_length * 0.5}" rpy="0 0 0" />
     </collision>
     <xacro:box_inertial_matrix m="${link_mass}" l="${link2_width}" w="${link2_width}" h="${link2_length}" />
@@ -107,5 +99,5 @@
     <parent link="link1" />
     <child link="link2" />
-    <origin xyz="0.0 0.0 ${link1_length}" rpy="0 0 0" />
+    <origin xyz="0.0 0.0 ${link1_length * 0.5 + link2_length * 0.5}" rpy="0 0 0" />
     <axis xyz="0 0 1" />
     <dynamics D="1" K="7000" damping="0.003" friction="0.0" mu_coulomb="0" mu_viscous="16" />
@@ -120,5 +112,4 @@
       </geometry>
       <material name="green"></material>
-      <origin xyz="${link3_length * 0.5} 0.0 0.0" rpy="0 0 0" />
     </visual>
     <collision>
@@ -126,5 +117,4 @@
         <box size="${link3_length} ${link3_width} ${link3_width}" />
       </geometry>
-      <origin xyz="${link3_length * 0.5} 0.0 0.0" rpy="0 0 0" />
     </collision>
     <xacro:box_inertial_matrix m="${link_mass}" l="${link3_length}" w="${link3_width}" h="${link3_width}" />
@@ -133,5 +123,5 @@
     <parent link="link2" />
     <child link="link3" />
-    <origin xyz="${link3_width * 0.5} 0.0 ${link2_length * 0.5}" rpy="0 0 0" />
+    <origin xyz="${link3_length * 0.5 + link2_width * 0.5} 0 0" rpy="0 0 0" />
     <axis xyz="0 0 1" />
     <limit lower="-${link2_length * 0.5 - link3_width * 0.5}" upper="${link2_length * 0.5 - link3_width * 0.5}" effort="10.0" velocity="1.0" />
@@ -147,5 +137,4 @@
       </geometry>
       <material name="red"></material>
-      <origin xyz="${link4_length * 0.5} 0.0 0.0" rpy="0 0 0" />
     </visual>
     <collision>
@@ -153,5 +142,4 @@
         <box size="${link4_length} ${link4_width} ${link4_width}" />
       </geometry>
-      <origin xyz="${link4_length * 0.5} 0.0 0.0" rpy="0 0 0" />
     </collision>
     <xacro:box_inertial_matrix m="${link_mass}" l="${link4_length}" w="${link4_width}" h="${link4_width}" />
@@ -160,5 +148,5 @@
     <parent link="link3" />
     <child link="link4" />
-    <origin xyz="${link3_length} 0.0 0.0" rpy="0 0 0" />
+    <origin xyz="${link3_length * 0.5 + link4_length * 0.5} 0.0 0.0" rpy="0 0 0" />
     <axis xyz="1 0 0" />
     <dynamics damping="0.7" friction="0.0" />

File: src/arm_robot/model/arm_robot.xacro (robot description, xacro)
@@ -1,4 +1,4 @@
 <robot xmlns:xacro="http://www.ros.org/wiki/xacro" name="robot">
-  <xacro:property name="transparency" value="0.8" />
+  <xacro:property name="transparency" value="0.5" />
   <xacro:include filename="$(find arm_robot)/model/util/util.xacro" />
   <!-- ========================= -->
@@ -6,9 +6,9 @@
   <!-- ========================= -->
   <xacro:property name="link0_length" value="10.0" />
-  <xacro:property name="link0_width" value="0.1" />
+  <xacro:property name="link0_width" value="0.06" />
   <xacro:property name="link1_length" value="0.3" />
-  <xacro:property name="link1_width" value="0.1" />
+  <xacro:property name="link1_width" value="0.06" />
   <xacro:property name="link2_length" value="3.0" />
-  <xacro:property name="link2_width" value="0.1" />
+  <xacro:property name="link2_width" value="0.06" />
   <xacro:property name="link3_length" value="0.1" />
   <xacro:property name="link3_width" value="0.06" />

File: src/arm_robot/model/robot/robot.xacro (robot description, xacro)
@@ -25,5 +25,5 @@
     <parent link="link4" />
     <child link="base_link" />
-    <origin xyz="${link4_length - base_box_size * 0.5} ${base_box_size * 0.5 + link4_width * 0.5} 0.0" rpy="0 0 0" />
+    <origin xyz="${link4_length * 0.5 - base_box_size * 0.5} ${base_box_size * 0.5 + link4_width * 0.5} 0.0" rpy="0 0 0" />
     <axis xyz="0 1 0" />
   </joint>

Commit message: update arm prams

File: src/arm_robot/model/arm/arm.xacro (robot description, xacro)
@@ -48,5 +48,5 @@
     <axis xyz="0 1 0" />
     <limit lower="-${platform_width * 0.5 - link0_width * 0.5}" upper="${platform_width * 0.5 - link0_width * 0.5}" effort="10.0" velocity="1.0" />
-    <dynamics D="1" K="7000" damping="0.003" friction="0.0" mu_coulomb="0" mu_viscous="16" />
+    <xacro:joint-dynamic />
   </joint>
   <gazebo reference="link0">
@@ -75,5 +75,5 @@
     <axis xyz="1 0 0" />
     <limit lower="-${link0_length * 0.5 - link1_width * 0.5}" upper="${link0_length * 0.5 - link1_width * 0.5}" effort="10.0" velocity="1.0" />
-    <dynamics D="1" K="7000" damping="0.003" friction="0.0" mu_coulomb="0" mu_viscous="16" />
+    <xacro:joint-dynamic />
   </joint>
   <gazebo reference="link1">
@@ -101,5 +101,5 @@
     <origin xyz="0.0 0.0 ${link1_length * 0.5 + link2_length * 0.5}" rpy="0 0 0" />
     <axis xyz="0 0 1" />
-    <dynamics D="1" K="7000" damping="0.003" friction="0.0" mu_coulomb="0" mu_viscous="16" />
+    <xacro:joint-dynamic />
   </joint>
   <gazebo reference="link2">
@@ -126,5 +126,5 @@
     <axis xyz="0 0 1" />
     <limit lower="-${link2_length * 0.5 - link3_width * 0.5}" upper="${link2_length * 0.5 - link3_width * 0.5}" effort="10.0" velocity="1.0" />
-    <dynamics D="1" K="7000" damping="0.003" friction="0.0" mu_coulomb="0" mu_viscous="16" />
+    <xacro:joint-dynamic />
   </joint>
   <gazebo reference="link3">
@@ -150,6 +150,5 @@
     <origin xyz="${link3_length * 0.5 + link4_length * 0.5} 0.0 0.0" rpy="0 0 0" />
     <axis xyz="1 0 0" />
-    <dynamics damping="0.7" friction="0.0" />
-    <dynamics D="1" K="7000" damping="0.003" friction="0.0" mu_coulomb="0" mu_viscous="16" />
+    <xacro:joint-dynamic />
   </joint>
   <gazebo reference="link4">

File: src/arm_robot/model/robot/robot.xacro (robot description, xacro)
@@ -27,4 +27,5 @@
     <origin xyz="${link4_length * 0.5 - base_box_size * 0.5} ${base_box_size * 0.5 + link4_width * 0.5} 0.0" rpy="0 0 0" />
     <axis xyz="0 1 0" />
+    <xacro:joint-dynamic />
   </joint>
   <xacro:include filename="lidar.xacro" />

File: src/arm_robot/model/util/util.xacro (robot description, xacro)
@@ -58,3 +58,7 @@
     </gazebo>
   </xacro:macro>
+  <xacro:macro name="joint-dynamic">
+    <dynamics damping="0.5" friction="10.0" />
+    <dynamics D="1" K="7000" damping="0.003" friction="0.0" mu_coulomb="0" mu_viscous="16" />
+  </xacro:macro>
 </robot>

Commit message: update arm prams

File: src/arm_robot/model/arm/arm.xacro (robot description, xacro)
@@ -123,5 +123,5 @@
     <parent link="link2" />
     <child link="link3" />
-    <origin xyz="${link3_length * 0.5 + link2_width * 0.5} 0 0" rpy="0 0 0" />
+    <origin xyz="0 ${link3_width * 0.5 + link2_width * 0.5} 0" rpy="0 0 0" />
     <axis xyz="0 0 1" />
     <limit lower="-${link2_length * 0.5 - link3_width * 0.5}" upper="${link2_length * 0.5 - link3_width * 0.5}" effort="10.0" velocity="1.0" />

File: src/arm_robot/model/robot/robot.xacro (robot description, xacro)
@@ -25,5 +25,5 @@
     <parent link="link4" />
     <child link="base_link" />
-    <origin xyz="${link4_length * 0.5 - base_box_size * 0.5} ${base_box_size * 0.5 + link4_width * 0.5} 0.0" rpy="0 0 0" />
+    <origin xyz="${link4_length * 0.5 - base_box_size * 0.5} -${base_box_size * 0.5 + link4_width * 0.5} 0.0" rpy="0 0 0" />
     <axis xyz="0 1 0" />
     <xacro:joint-dynamic />

File: src/arm_robot/model/util/util.xacro (robot description, xacro)
@@ -59,6 +59,5 @@
   </xacro:macro>
   <xacro:macro name="joint-dynamic">
-    <dynamics damping="0.5" friction="10.0" />
-    <dynamics D="1" K="7000" damping="0.003" friction="0.0" mu_coulomb="0" mu_viscous="16" />
+    <dynamics D="1" K="7000" damping="0.003" friction="10.0" mu_coulomb="0" mu_viscous="16" />
   </xacro:macro>
 </robot>

Commit message: update arm prams

File: src/arm_robot/model/arm/arm.xacro (robot description, xacro)
@@ -155,3 +155,27 @@
     <material>Gazebo/Red</material>
   </gazebo>
+  <link name="link5">
+    <visual>
+      <geometry>
+        <box size="${link4_length} ${link4_width} ${link4_width}" />
+      </geometry>
+      <material name="red"></material>
+    </visual>
+    <collision>
+      <geometry>
+        <box size="${link4_length} ${link4_width} ${link4_width}" />
+      </geometry>
+    </collision>
+    <xacro:box_inertial_matrix m="${link_mass}" l="${link4_length}" w="${link4_width}" h="${link4_width}" />
+  </link>
+  <joint name="link5_to_link3" type="fixed">
+    <parent link="link3" />
+    <child link="link5" />
+    <origin xyz="-${link3_length * 0.5 + link4_length * 0.5} 0.0 0.0" rpy="0 0 0" />
+    <axis xyz="1 0 0" />
+    <xacro:joint-dynamic />
+  </joint>
+  <gazebo reference="link5">
+    <material>Gazebo/Red</material>
+  </gazebo>
 </robot>

File: src/arm_robot/model/arm_robot.xacro (robot description, xacro)
@@ -15,6 +15,4 @@
   <xacro:property name="link4_length" value="0.15" />
   <xacro:property name="link4_width" value="0.06" />
-  <xacro:property name="link5_length" value="0.1" />
-  <xacro:property name="link5_width" value="0.06" />
   <xacro:property name="platform_width" value="10.0" />
   <xacro:property name="platform_length" value="0.1" />

Commit message: update arm prams

File: src/arm_robot/model/arm/arm.xacro (robot description, xacro)
@@ -155,27 +155,3 @@
     <material>Gazebo/Red</material>
   </gazebo>
-  <link name="link5">
-    <visual>
-      <geometry>
-        <box size="${link4_length} ${link4_width} ${link4_width}" />
-      </geometry>
-      <material name="red"></material>
-    </visual>
-    <collision>
-      <geometry>
-        <box size="${link4_length} ${link4_width} ${link4_width}" />
-      </geometry>
-    </collision>
-    <xacro:box_inertial_matrix m="${link_mass}" l="${link4_length}" w="${link4_width}" h="${link4_width}" />
-  </link>
-  <joint name="link5_to_link3" type="fixed">
-    <parent link="link3" />
-    <child link="link5" />
-    <origin xyz="-${link3_length * 0.5 + link4_length * 0.5} 0.0 0.0" rpy="0 0 0" />
-    <axis xyz="1 0 0" />
-    <xacro:joint-dynamic />
-  </joint>
-  <gazebo reference="link5">
-    <material>Gazebo/Red</material>
-  </gazebo>
 </robot>

File: src/arm_robot/model/arm_robot.xacro (robot description, xacro)
@@ -9,5 +9,5 @@
   <xacro:property name="link1_length" value="0.06" />
   <xacro:property name="link1_width" value="0.06" />
-  <xacro:property name="link2_length" value="3.0" />
+  <xacro:property name="link2_length" value="2.0" />
   <xacro:property name="link2_width" value="0.06" />
   <xacro:property name="link3_length" value="0.06" />

Commit message: split link mass

File: src/arm_robot/model/arm/arm.xacro (robot description, xacro)
@@ -40,5 +40,5 @@
       </geometry>
     </collision>
-    <xacro:box_inertial_matrix m="${link_mass}" l="${link0_length}" w="${link0_width}" h="${link0_width}" />
+    <xacro:box_inertial_matrix m="${link0_mass}" l="${link0_length}" w="${link0_width}" h="${link0_width}" />
   </link>
   <joint name="link0_to_platform" type="prismatic">
@@ -67,5 +67,5 @@
       </geometry>
     </collision>
-    <xacro:box_inertial_matrix m="${link_mass}" l="${link1_width}" w="${link1_width}" h="${link1_length}" />
+    <xacro:box_inertial_matrix m="${link1_mass}" l="${link1_width}" w="${link1_width}" h="${link1_length}" />
   </link>
   <joint name="link1_to_link0" type="prismatic">
@@ -94,5 +94,5 @@
       </geometry>
     </collision>
-    <xacro:box_inertial_matrix m="${link_mass}" l="${link2_width}" w="${link2_width}" h="${link2_length}" />
+    <xacro:box_inertial_matrix m="${link2_mass}" l="${link2_width}" w="${link2_width}" h="${link2_length}" />
   </link>
   <joint name="link2_to_link1" type="continuous">
@@ -118,5 +118,5 @@
       </geometry>
     </collision>
-    <xacro:box_inertial_matrix m="${link_mass}" l="${link3_length}" w="${link3_width}" h="${link3_width}" />
+    <xacro:box_inertial_matrix m="${link3_mass}" l="${link3_length}" w="${link3_width}" h="${link3_width}" />
   </link>
   <joint name="link3_to_link2" type="prismatic">
@@ -143,5 +143,5 @@
       </geometry>
     </collision>
-    <xacro:box_inertial_matrix m="${link_mass}" l="${link4_length}" w="${link4_width}" h="${link4_width}" />
+    <xacro:box_inertial_matrix m="${link4_mass}" l="${link4_length}" w="${link4_width}" h="${link4_width}" />
   </link>
   <joint name="link4_to_link3" type="continuous">

File: src/arm_robot/model/arm_robot.xacro (robot description, xacro)
@@ -18,5 +18,9 @@
   <xacro:property name="platform_length" value="0.1" />
   <xacro:property name="platform_mass" value="100.0" />
-  <xacro:property name="link_mass" value="0.1" />
+  <xacro:property name="link0_mass" value="10" />
+  <xacro:property name="link1_mass" value="0.3" />
+  <xacro:property name="link2_mass" value="3" />
+  <xacro:property name="link3_mass" value="0.1" />
+  <xacro:property name="link4_mass" value="0.15" />
   <!-- ========================= -->
   <!-- |    for robot params   | -->

Commit message: split link mass

File: src/arm_robot/model/arm/arm.xacro (robot description, xacro)
@@ -54,5 +54,5 @@
   </gazebo>
   <link name="link1">
-    <visual>
+    <!-- <visual>
       <geometry>
         <box size="${link1_width} ${link1_width} ${link1_length}" />
@@ -61,5 +61,5 @@
         <color rgba="0 1.0 0 ${transparency}" />
       </material>
-    </visual>
+    </visual> -->
     <collision>
       <geometry>
@@ -81,5 +81,5 @@
   </gazebo>
   <link name="link2">
-    <visual>
+    <!-- <visual>
       <geometry>
         <box size="${link2_width} ${link2_width} ${link2_length}" />
@@ -88,5 +88,5 @@
         <color rgba="1.0 0 0 ${transparency}" />
       </material>
-    </visual>
+    </visual> -->
     <collision>
       <geometry>
@@ -107,10 +107,10 @@
   </gazebo>
   <link name="link3">
-    <visual>
+    <!-- <visual>
       <geometry>
         <box size="${link3_length} ${link3_width} ${link3_width}" />
       </geometry>
       <material name="green"></material>
-    </visual>
+    </visual> -->
     <collision>
       <geometry>
@@ -132,10 +132,10 @@
   </gazebo>
   <link name="link4">
-    <visual>
+    <!-- <visual>
       <geometry>
         <box size="${link4_length} ${link4_width} ${link4_width}" />
       </geometry>
       <material name="red"></material>
-    </visual>
+    </visual> -->
     <collision>
       <geometry>
