Commit message: remove collision and visual

File: src/arm_robot/model/arm/arm.xacro (robot description, xacro)
@@ -2,5 +2,5 @@
   <link name="platform_footprint"></link>
   <link name="platform">
-    <visual>
+    <!-- <visual>
       <geometry>
         <box size="${platform_width} ${platform_width} ${platform_length}" />
@@ -9,5 +9,5 @@
         <color rgba="0 0 1.0 ${transparency}" />
       </material>
-    </visual>
+    </visual> -->
     <collision>
       <geometry>
@@ -27,5 +27,5 @@
   </gazebo>
   <link name="link0">
-    <visual>
+    <!-- <visual>
       <geometry>
         <box size="${link0_length} ${link0_width} ${link0_width}" />
@@ -34,9 +34,10 @@
         <color rgba="1.0 0 0 ${transparency}" />
       </material>
-    </visual>
+    </visual> -->
     <collision>
       <geometry>
         <box size="${link0_length} ${link0_width} ${link0_width}" />
       </geometry>
+      <xacro:remove-collision />
     </collision>
     <xacro:box_inertial_matrix m="${link0_mass}" l="${link0_length}" w="${link0_width}" h="${link0_width}" />
@@ -66,4 +67,5 @@
         <box size="${link1_width} ${link1_width} ${link1_length}" />
       </geometry>
+      <xacro:remove-collision />
     </collision>
     <xacro:box_inertial_matrix m="${link1_mass}" l="${link1_width}" w="${link1_width}" h="${link1_length}" />
@@ -93,4 +95,5 @@
         <box size="${link2_width} ${link2_width} ${link2_length}" />
       </geometry>
+      <xacro:remove-collision />
     </collision>
     <xacro:box_inertial_matrix m="${link2_mass}" l="${link2_width}" w="${link2_width}" h="${link2_length}" />
@@ -117,4 +120,5 @@
         <box size="${link3_length} ${link3_width} ${link3_width}" />
       </geometry>
+      <xacro:remove-collision />
     </collision>
     <xacro:box_inertial_matrix m="${link3_mass}" l="${link3_length}" w="${link3_width}" h="${link3_width}" />
@@ -142,4 +146,5 @@
         <box size="${link4_length} ${link4_width} ${link4_width}" />
       </geometry>
+      <xacro:remove-collision />
     </collision>
     <xacro:box_inertial_matrix m="${link4_mass}" l="${link4_length}" w="${link4_width}" h="${link4_width}" />

File: src/arm_robot/model/arm_robot.xacro (robot description, xacro)
@@ -16,5 +16,5 @@
   <xacro:property name="link4_width" value="0.06" />
   <xacro:property name="platform_width" value="10.0" />
-  <xacro:property name="platform_length" value="0.1" />
+  <xacro:property name="platform_length" value="0.001" />
   <xacro:property name="platform_mass" value="100.0" />
   <xacro:property name="link0_mass" value="10" />

File: src/arm_robot/model/robot/camera.xacro (robot description, xacro)
@@ -15,5 +15,5 @@
         <box size="${camera_box_size} ${camera_box_size} ${camera_box_size}" />
       </geometry>
-      <origin xyz="0.0 0.0 0.0" rpy="0.0 0.0 0.0" />
+      <xacro:remove-collision />
     </collision>
     <xacro:box_inertial_matrix m="${camera_mass}" l="${camera_box_size}" w="${camera_box_size}" h="${camera_box_size}" />

File: src/arm_robot/model/robot/imu.xacro (robot description, xacro)
@@ -15,5 +15,5 @@
         <box size="${imu_box_size} ${imu_box_size} ${imu_box_size}" />
       </geometry>
-      <origin xyz="0.0 0.0 0.0" rpy="0.0 0.0 0.0" />
+      <xacro:remove-collision />
     </collision>
     <xacro:box_inertial_matrix m="${imu_mass}" l="${imu_box_size}" w="${imu_box_size}" h="${imu_box_size}" />

File: src/arm_robot/model/robot/lidar.xacro (robot description, xacro)
@@ -15,5 +15,5 @@
         <cylinder radius="${arm_cylinder_radius}" length="${arm_cylinder_length}" />
       </geometry>
-      <origin xyz="0.0 0.0 0.0" rpy="0.0 0.0 0.0" />
+      <xacro:remove-collision />
     </collision>
     <xacro:cylinder_inertial_matrix m="${arm_mass}" r="${arm_cylinder_radius}" h="${arm_cylinder_length}" />
@@ -44,5 +44,5 @@
         <cylinder radius="${lidar_cylinder_radius}" length="${lidar_cylinder_length}" />
       </geometry>
-      <origin xyz="0.0 0.0 0.0" rpy="0.0 0.0 0.0" />
+      <xacro:remove-collision />
     </collision>
     <xacro:cylinder_inertial_matrix m="${lidar_mass}" r="${lidar_cylinder_radius}" h="${lidar_cylinder_length}" />

File: src/arm_robot/model/robot/robot.xacro (robot description, xacro)
@@ -14,5 +14,5 @@
         <box size="${base_box_size} ${base_box_size} ${base_box_size}" />
       </geometry>
-      <origin xyz="0.0 0.0 0.0" rpy="0.0 0.0 0.0" />
+      <xacro:remove-collision />
     </collision>
     <xacro:box_inertial_matrix m="${base_mass}" l="${base_box_size}" w="${base_box_size}" h="${base_box_size}" />

File: src/arm_robot/model/util/util.xacro (robot description, xacro)
@@ -61,3 +61,6 @@
     <dynamics D="1" K="7000" damping="0.003" friction="10.0" mu_coulomb="0" mu_viscous="16" />
   </xacro:macro>
+  <xacro:macro name="remove-collision">
+    <origin xyz="0.0 0.0 10000.0" rpy="0 0 0" />
+  </xacro:macro>
 </robot>

Commit message: remove collision and visual

File: src/arm_robot/model/arm/arm.xacro (robot description, xacro)
@@ -35,10 +35,5 @@
       </material>
     </visual> -->
-    <collision>
-      <geometry>
-        <box size="${link0_length} ${link0_width} ${link0_width}" />
-      </geometry>
-      <xacro:remove-collision />
-    </collision>
+    <xacro:remove-collision />
     <xacro:box_inertial_matrix m="${link0_mass}" l="${link0_length}" w="${link0_width}" h="${link0_width}" />
   </link>
@@ -63,10 +58,5 @@
       </material>
     </visual> -->
-    <collision>
-      <geometry>
-        <box size="${link1_width} ${link1_width} ${link1_length}" />
-      </geometry>
-      <xacro:remove-collision />
-    </collision>
+    <xacro:remove-collision />
     <xacro:box_inertial_matrix m="${link1_mass}" l="${link1_width}" w="${link1_width}" h="${link1_length}" />
   </link>
@@ -91,10 +81,5 @@
       </material>
     </visual> -->
-    <collision>
-      <geometry>
-        <box size="${link2_width} ${link2_width} ${link2_length}" />
-      </geometry>
-      <xacro:remove-collision />
-    </collision>
+    <xacro:remove-collision />
     <xacro:box_inertial_matrix m="${link2_mass}" l="${link2_width}" w="${link2_width}" h="${link2_length}" />
   </link>
@@ -116,10 +101,5 @@
       <material name="green"></material>
     </visual> -->
-    <collision>
-      <geometry>
-        <box size="${link3_length} ${link3_width} ${link3_width}" />
-      </geometry>
-      <xacro:remove-collision />
-    </collision>
+    <xacro:remove-collision />
     <xacro:box_inertial_matrix m="${link3_mass}" l="${link3_length}" w="${link3_width}" h="${link3_width}" />
   </link>
@@ -142,10 +122,5 @@
       <material name="red"></material>
     </visual> -->
-    <collision>
-      <geometry>
-        <box size="${link4_length} ${link4_width} ${link4_width}" />
-      </geometry>
-      <xacro:remove-collision />
-    </collision>
+    <xacro:remove-collision />
     <xacro:box_inertial_matrix m="${link4_mass}" l="${link4_length}" w="${link4_width}" h="${link4_width}" />
   </link>

File: src/arm_robot/model/robot/camera.xacro (robot description, xacro)
@@ -11,10 +11,5 @@
       </material>
     </visual>
-    <collision>
-      <geometry>
-        <box size="${camera_box_size} ${camera_box_size} ${camera_box_size}" />
-      </geometry>
-      <xacro:remove-collision />
-    </collision>
+    <xacro:remove-collision />
     <xacro:box_inertial_matrix m="${camera_mass}" l="${camera_box_size}" w="${camera_box_size}" h="${camera_box_size}" />
   </link>

File: src/arm_robot/model/robot/imu.xacro (robot description, xacro)
@@ -11,10 +11,5 @@
       </material>
     </visual>
-    <collision>
-      <geometry>
-        <box size="${imu_box_size} ${imu_box_size} ${imu_box_size}" />
-      </geometry>
-      <xacro:remove-collision />
-    </collision>
+    <xacro:remove-collision />
     <xacro:box_inertial_matrix m="${imu_mass}" l="${imu_box_size}" w="${imu_box_size}" h="${imu_box_size}" />
   </link>

File: src/arm_robot/model/robot/lidar.xacro (robot description, xacro)
@@ -11,10 +11,5 @@
       </material>
     </visual>
-    <collision>
-      <geometry>
-        <cylinder radius="${arm_cylinder_radius}" length="${arm_cylinder_length}" />
-      </geometry>
-      <xacro:remove-collision />
-    </collision>
+    <xacro:remove-collision />
     <xacro:cylinder_inertial_matrix m="${arm_mass}" r="${arm_cylinder_radius}" h="${arm_cylinder_length}" />
   </link>
@@ -40,10 +35,5 @@
       </material>
     </visual>
-    <collision>
-      <geometry>
-        <cylinder radius="${lidar_cylinder_radius}" length="${lidar_cylinder_length}" />
-      </geometry>
-      <xacro:remove-collision />
-    </collision>
+    <xacro:remove-collision />
     <xacro:cylinder_inertial_matrix m="${lidar_mass}" r="${lidar_cylinder_radius}" h="${lidar_cylinder_length}" />
   </link>

File: src/arm_robot/model/robot/robot.xacro (robot description, xacro)
@@ -10,10 +10,5 @@
       </material>
     </visual>
-    <collision>
-      <geometry>
-        <box size="${base_box_size} ${base_box_size} ${base_box_size}" />
-      </geometry>
-      <xacro:remove-collision />
-    </collision>
+    <xacro:remove-collision />
     <xacro:box_inertial_matrix m="${base_mass}" l="${base_box_size}" w="${base_box_size}" h="${base_box_size}" />
   </link>

File: src/arm_robot/model/util/util.xacro (robot description, xacro)
@@ -62,5 +62,10 @@
   </xacro:macro>
   <xacro:macro name="remove-collision">
-    <origin xyz="0.0 0.0 10000.0" rpy="0 0 0" />
+    <collision>
+      <geometry>
+        <box size="0.001 0.001 0.001" />
+      </geometry>
+      <origin xyz="0.0 0.0 1000.0" rpy="0 0 0" />
+    </collision>
   </xacro:macro>
 </robot>

Commit message: add visula and collision

File: src/arm_robot/model/arm/arm.xacro (robot description, xacro)
@@ -2,5 +2,5 @@
   <link name="platform_footprint"></link>
   <link name="platform">
-    <!-- <visual>
+    <visual>
       <geometry>
         <box size="${platform_width} ${platform_width} ${platform_length}" />
@@ -9,5 +9,5 @@
         <color rgba="0 0 1.0 ${transparency}" />
       </material>
-    </visual> -->
+    </visual>
     <collision>
       <geometry>
@@ -27,5 +27,5 @@
   </gazebo>
   <link name="link0">
-    <!-- <visual>
+    <visual>
       <geometry>
         <box size="${link0_length} ${link0_width} ${link0_width}" />
@@ -34,6 +34,10 @@
         <color rgba="1.0 0 0 ${transparency}" />
       </material>
-    </visual> -->
-    <xacro:remove-collision />
+    </visual>
+    <collision>
+      <geometry>
+        <box size="${link0_length} ${link0_width} ${link0_width}" />
+      </geometry>
+    </collision>
     <xacro:box_inertial_matrix m="${link0_mass}" l="${link0_length}" w="${link0_width}" h="${link0_width}" />
   </link>
@@ -50,5 +54,5 @@
   </gazebo>
   <link name="link1">
-    <!-- <visual>
+    <visual>
       <geometry>
         <box size="${link1_width} ${link1_width} ${link1_length}" />
@@ -57,6 +61,10 @@
         <color rgba="0 1.0 0 ${transparency}" />
       </material>
-    </visual> -->
-    <xacro:remove-collision />
+    </visual>
+    <collision>
+      <geometry>
+        <box size="${link1_width} ${link1_width} ${link1_length}" />
+      </geometry>
+    </collision>
     <xacro:box_inertial_matrix m="${link1_mass}" l="${link1_width}" w="${link1_width}" h="${link1_length}" />
   </link>
@@ -73,5 +81,5 @@
   </gazebo>
   <link name="link2">
-    <!-- <visual>
+    <visual>
       <geometry>
         <box size="${link2_width} ${link2_width} ${link2_length}" />
@@ -80,6 +88,10 @@
         <color rgba="1.0 0 0 ${transparency}" />
       </material>
-    </visual> -->
-    <xacro:remove-collision />
+    </visual>
+    <collision>
+      <geometry>
+        <box size="${link2_width} ${link2_width} ${link2_length}" />
+      </geometry>
+    </collision>
     <xacro:box_inertial_matrix m="${link2_mass}" l="${link2_width}" w="${link2_width}" h="${link2_length}" />
   </link>
@@ -95,11 +107,15 @@
   </gazebo>
   <link name="link3">
-    <!-- <visual>
+    <visual>
       <geometry>
         <box size="${link3_length} ${link3_width} ${link3_width}" />
       </geometry>
       <material name="green"></material>
-    </visual> -->
-    <xacro:remove-collision />
+    </visual>
+    <collision>
+      <geometry>
+        <box size="${link3_length} ${link3_width} ${link3_width}" />
+      </geometry>
+    </collision>
     <xacro:box_inertial_matrix m="${link3_mass}" l="${link3_length}" w="${link3_width}" h="${link3_width}" />
   </link>
@@ -116,11 +132,15 @@
   </gazebo>
   <link name="link4">
-    <!-- <visual>
+    <visual>
       <geometry>
         <box size="${link4_length} ${link4_width} ${link4_width}" />
       </geometry>
       <material name="red"></material>
-    </visual> -->
-    <xacro:remove-collision />
+    </visual>
+    <collision>
+      <geometry>
+        <box size="${link4_length} ${link4_width} ${link4_width}" />
+      </geometry>
+    </collision>
     <xacro:box_inertial_matrix m="${link4_mass}" l="${link4_length}" w="${link4_width}" h="${link4_width}" />
   </link>

File: src/arm_robot/model/robot/camera.xacro (robot description, xacro)
@@ -11,5 +11,9 @@
       </material>
     </visual>
-    <xacro:remove-collision />
+    <collision>
+      <geometry>
+        <box size="${camera_box_size} ${camera_box_size} ${camera_box_size}" />
+      </geometry>
+    </collision>
     <xacro:box_inertial_matrix m="${camera_mass}" l="${camera_box_size}" w="${camera_box_size}" h="${camera_box_size}" />
   </link>

File: src/arm_robot/model/robot/imu.xacro (robot description, xacro)
@@ -11,5 +11,9 @@
       </material>
     </visual>
-    <xacro:remove-collision />
+    <collision>
+      <geometry>
+        <box size="${imu_box_size} ${imu_box_size} ${imu_box_size}" />
+      </geometry>
+    </collision>
     <xacro:box_inertial_matrix m="${imu_mass}" l="${imu_box_size}" w="${imu_box_size}" h="${imu_box_size}" />
   </link>

File: src/arm_robot/model/robot/lidar.xacro (robot description, xacro)
@@ -11,5 +11,9 @@
       </material>
     </visual>
-    <xacro:remove-collision />
+    <collision>
+      <geometry>
+        <cylinder radius="${arm_cylinder_radius}" length="${arm_cylinder_length}" />
+      </geometry>
+    </collision>
     <xacro:cylinder_inertial_matrix m="${arm_mass}" r="${arm_cylinder_radius}" h="${arm_cylinder_length}" />
   </link>
@@ -35,5 +39,9 @@
       </material>
     </visual>
-    <xacro:remove-collision />
+    <collision>
+      <geometry>
+        <cylinder radius="${lidar_cylinder_radius}" length="${lidar_cylinder_length}" />
+      </geometry>
+    </collision>
     <xacro:cylinder_inertial_matrix m="${lidar_mass}" r="${lidar_cylinder_radius}" h="${lidar_cylinder_length}" />
   </link>

File: src/arm_robot/model/robot/robot.xacro (robot description, xacro)
@@ -10,5 +10,9 @@
       </material>
     </visual>
-    <xacro:remove-collision />
+    <collision>
+      <geometry>
+        <box size="${base_box_size} ${base_box_size} ${base_box_size}" />
+      </geometry>
+    </collision>
     <xacro:box_inertial_matrix m="${base_mass}" l="${base_box_size}" w="${base_box_size}" h="${base_box_size}" />
   </link>

File: src/arm_robot/model/util/util.xacro (robot description, xacro)
@@ -61,11 +61,3 @@
     <dynamics D="1" K="7000" damping="0.003" friction="10.0" mu_coulomb="0" mu_viscous="16" />
   </xacro:macro>
-  <xacro:macro name="remove-collision">
-    <collision>
-      <geometry>
-        <box size="0.001 0.001 0.001" />
-      </geometry>
-      <origin xyz="0.0 0.0 1000.0" rpy="0 0 0" />
-    </collision>
-  </xacro:macro>
 </robot>

Commit message: good

File: src/arm_robot/model/arm/arm.xacro (robot description, xacro)
@@ -47,5 +47,5 @@
     <origin xyz="0.0 0.0 ${platform_length * 0.5 + link0_width * 0.5}" rpy="0 0 0" />
     <axis xyz="0 1 0" />
-    <limit lower="-${platform_width * 0.5 - link0_width * 0.5}" upper="${platform_width * 0.5 - link0_width * 0.5}" effort="10.0" velocity="1.0" />
+    <limit lower="-${platform_width * 0.5 - link0_width * 0.5}" upper="${platform_width * 0.5 - link0_width * 0.5}" effort="10000000.0" velocity="1000000.0" />
     <xacro:joint-dynamic />
   </joint>
@@ -74,5 +74,5 @@
     <origin xyz="0.0 0.0 ${link0_width * 0.5 + link1_length * 0.5}" rpy="0 0 0" />
     <axis xyz="1 0 0" />
-    <limit lower="-${link0_length * 0.5 - link1_width * 0.5}" upper="${link0_length * 0.5 - link1_width * 0.5}" effort="10.0" velocity="1.0" />
+    <limit lower="-${link0_length * 0.5 - link1_width * 0.5}" upper="${link0_length * 0.5 - link1_width * 0.5}" effort="10000000.0" velocity="1000000.0" />
     <xacro:joint-dynamic />
   </joint>
@@ -125,5 +125,5 @@
     <origin xyz="0 ${link3_width * 0.5 + link2_width * 0.5} 0" rpy="0 0 0" />
     <axis xyz="0 0 1" />
-    <limit lower="-${link2_length * 0.5 - link3_width * 0.5}" upper="${link2_length * 0.5 - link3_width * 0.5}" effort="10.0" velocity="1.0" />
+    <limit lower="-${link2_length * 0.5 - link3_width * 0.5}" upper="${link2_length * 0.5 - link3_width * 0.5}" effort="10000000.0" velocity="1000000.0" />
     <xacro:joint-dynamic />
   </joint>

File: src/arm_robot/model/arm_robot.xacro (robot description, xacro)
@@ -17,10 +17,10 @@
   <xacro:property name="platform_width" value="10.0" />
   <xacro:property name="platform_length" value="0.001" />
-  <xacro:property name="platform_mass" value="100.0" />
-  <xacro:property name="link0_mass" value="10" />
-  <xacro:property name="link1_mass" value="0.3" />
-  <xacro:property name="link2_mass" value="3" />
-  <xacro:property name="link3_mass" value="0.1" />
-  <xacro:property name="link4_mass" value="0.15" />
+  <xacro:property name="platform_mass" value="1000000.0" />
+  <xacro:property name="link0_mass" value="50000" />
+  <xacro:property name="link1_mass" value="50000" />
+  <xacro:property name="link2_mass" value="100" />
+  <xacro:property name="link3_mass" value="10" />
+  <xacro:property name="link4_mass" value="0.1" />
   <!-- ========================= -->
   <!-- |    for robot params   | -->

Commit message: update

File: src/arm_robot/model/arm/arm.xacro (robot description, xacro)
@@ -123,5 +123,5 @@
     <parent link="link2" />
     <child link="link3" />
-    <origin xyz="0 ${link3_width * 0.5 + link2_width * 0.5} 0" rpy="0 0 0" />
+    <origin xyz="0 0 0" rpy="0 0 0" />
     <axis xyz="0 0 1" />
     <limit lower="-${link2_length * 0.5 - link3_width * 0.5}" upper="${link2_length * 0.5 - link3_width * 0.5}" effort="10000000.0" velocity="1000000.0" />

Commit message: change structure

File: src/arm_robot/model/arm/arm.xacro (robot description, xacro)
@@ -72,5 +72,5 @@
     <parent link="link0" />
     <child link="link1" />
-    <origin xyz="0.0 0.0 ${link0_width * 0.5 + link1_length * 0.5}" rpy="0 0 0" />
+    <origin xyz="0.0 0.0 ${0.5 * link1_length}" rpy="0 0 0" />
     <axis xyz="1 0 0" />
     <limit lower="-${link0_length * 0.5 - link1_width * 0.5}" upper="${link0_length * 0.5 - link1_width * 0.5}" effort="10000000.0" velocity="1000000.0" />
@@ -125,5 +125,5 @@
     <origin xyz="0 0 0" rpy="0 0 0" />
     <axis xyz="0 0 1" />
-    <limit lower="-${link2_length * 0.5 - link3_width * 0.5}" upper="${link2_length * 0.5 - link3_width * 0.5}" effort="10000000.0" velocity="1000000.0" />
+    <limit lower="-${link2_length * 0.5 - link3_width * 3.0}" upper="${link2_length * 0.5 - link3_width * 0.5}" effort="10000000.0" velocity="1000000.0" />
     <xacro:joint-dynamic />
   </joint>

File: src/arm_robot/model/arm_robot.xacro (robot description, xacro)
@@ -7,5 +7,5 @@
   <xacro:property name="link0_length" value="10.0" />
   <xacro:property name="link0_width" value="0.06" />
-  <xacro:property name="link1_length" value="0.2" />
+  <xacro:property name="link1_length" value="0.06" />
   <xacro:property name="link1_width" value="0.06" />
   <xacro:property name="link2_length" value="3.0" />
@@ -13,8 +13,8 @@
   <xacro:property name="link3_length" value="0.1" />
   <xacro:property name="link3_width" value="0.06" />
-  <xacro:property name="link4_length" value="0.15" />
+  <xacro:property name="link4_length" value="0.2" />
   <xacro:property name="link4_width" value="0.06" />
   <xacro:property name="platform_width" value="10.0" />
-  <xacro:property name="platform_length" value="0.001" />
+  <xacro:property name="platform_length" value="0.06" />
   <xacro:property name="platform_mass" value="1000000.0" />
   <xacro:property name="link0_mass" value="50000" />

File: src/arm_robot/model/robot/robot.xacro (robot description, xacro)
@@ -24,5 +24,5 @@
     <parent link="link4" />
     <child link="base_link" />
-    <origin xyz="${link4_length * 0.5 - base_box_size * 0.5} -${base_box_size * 0.5 + link4_width * 0.5} 0.0" rpy="0 0 0" />
+    <origin xyz="0.0 -${base_box_size * 0.5 + link4_width * 0.5} 0.0" rpy="0 0 0" />
     <axis xyz="0 1 0" />
     <xacro:joint-dynamic />
