Commit message: everything is fine

File: src/scene/model/urdf/sim-robot.urdf (robot description, URDF)
Before this commit: robot sim-robot, 5 links, 4 joints
Links:
- added link arm, mass 0.01; collision cylinder length=0.1 radius=0.01; visual cylinder length=0.1 radius=0.01
- added link back_support_wheel, mass 2.0; collision sphere radius=0.015; visual sphere radius=0.015
- added link front_support_wheel, mass 2.0; collision sphere radius=0.015; visual sphere radius=0.015
- added link left_wheel, mass 2.0; collision cylinder length=0.04 radius=0.08; visual cylinder length=0.04 radius=0.08
- added link right_wheel, mass 2.0; collision cylinder length=0.04 radius=0.08; visual cylinder length=0.04 radius=0.08
- link base_footprint: geometry visual box size=0.001 0.001 0.001
- link base_link: mass 20.0 -> 0.5; geometry collision box size=0.3 0.3 0.3; visual box size=0.3 0.3 0.3
- link camera: mass 1.0 -> 0.01; geometry collision box size=0.06 0.06 0.06; visual box size=0.06 0.06 0.06
- link imu: mass 1.0 -> 0.01; geometry collision box size=0.06 0.06 0.06; visual box size=0.06 0.06 0.06
- link lidar: mass 5.0 -> 0.02; geometry collision cylinder length=0.05 radius=0.05; visual cylinder length=0.05 radius=0.05
Joints:
- removed joint lidar_to_base_link
- added joint arm_to_base_link: type fixed, parent base_link, child arm, origin xyz=0.0 0.0 0.2 rpy=0.0 0.0 0.0, axis 0.0 0.0 1.0
- added joint back_support_wheel_to_base_link: type continuous, parent base_link, child back_support_wheel, origin xyz=-0.135 0.0 -0.16499999999999998, axis 1 1 1
- added joint front_support_wheel_to_base_link: type continuous, parent base_link, child front_support_wheel, origin xyz=0.135 0.0 -0.16499999999999998, axis 1 1 1
- added joint left_wheel_to_base_link: type continuous, parent base_link, child left_wheel, origin xyz=0.0 0.15 -0.09999999999999999, axis 0 1 0
- added joint lidar_to_arm: type fixed, parent arm, child lidar, origin xyz=0.0 0.0 0.07500000000000001 rpy=0.0 0.0 0.0, axis 0.0 0.0 1.0
- added joint right_wheel_to_base_link: type continuous, parent base_link, child right_wheel, origin xyz=0.0 -0.15 -0.09999999999999999, axis 0 1 0
- joint base_to_foot: origin xyz=0.0 0.0 0.1 rpy=0.0 0.0 0.0 -> xyz=0.0 0.0 0.18 rpy=0.0 0.0 0.0
- joint camera_to_base_link: origin xyz=0.15000000000000002 0.0 0.0 rpy=0.0 0.0 0.0 -> xyz=0.18 0.0 0.0 rpy=0.0 0.0 0.0
- joint imu_to_base_link: origin xyz=0.0 0.15000000000000002 0.0 rpy=0.0 0.0 0.0 -> xyz=-0.18 0.0 0.0 rpy=0.0 0.0 0.0

File: src/scene/model/xacro/sensor-laser.xacro (robot description, xacro)
@@ -34,4 +34,8 @@
         <topicName>/sim_lidar/scan</topicName>
         <frameName>/lidar</frameName>
+        <organize_cloud>true</organize_cloud>
+        <min_range>0.10</min_range>
+        <max_range>30.0</max_range>
+        <gaussianNoise>0.0</gaussianNoise>
       </plugin>
     </sensor>

Commit message: change lunch file name and

File: src/scene/model/urdf/sim-robot.urdf (robot description, URDF)
Before this commit: robot sim-robot, 10 links, 9 joints
Links:
- link back_support_wheel: mass 2.0 -> 0.3
- link front_support_wheel: mass 2.0 -> 0.3
- link left_wheel: mass 2.0 -> 0.3
- link right_wheel: mass 2.0 -> 0.3

Commit message: update

File: src/scene/model/urdf/sim-robot.urdf (robot description, URDF)
Before this commit: robot sim-robot, 10 links, 9 joints
Links:
- removed link back_support_wheel
- removed link front_support_wheel
- removed link left_wheel
- removed link right_wheel
- link arm: geometry collision cylinder length=0.05 radius=0.01; visual cylinder length=0.05 radius=0.01
- link base_link: geometry collision box size=0.1 0.1 0.1; visual box size=0.1 0.1 0.1
Joints:
- removed joint back_support_wheel_to_base_link
- removed joint front_support_wheel_to_base_link
- removed joint left_wheel_to_base_link
- removed joint right_wheel_to_base_link
- joint arm_to_base_link: origin xyz=0.0 0.0 0.2 rpy=0.0 0.0 0.0 -> xyz=0.0 0.0 0.07500000000000001 rpy=0.0 0.0 0.0
- joint base_to_foot: origin xyz=0.0 0.0 0.18 rpy=0.0 0.0 0.0 -> xyz=0.0 0.0 0.08 rpy=0.0 0.0 0.0
- joint camera_to_base_link: origin xyz=0.18 0.0 0.0 rpy=0.0 0.0 0.0 -> xyz=0.08 0.0 0.0 rpy=0.0 0.0 0.0
- joint imu_to_base_link: origin xyz=-0.18 0.0 0.0 rpy=0.0 0.0 0.0 -> xyz=-0.08 0.0 0.0 rpy=0.0 0.0 0.0
- joint lidar_to_arm: origin xyz=0.0 0.0 0.07500000000000001 rpy=0.0 0.0 0.0 -> xyz=0.0 0.0 0.05 rpy=0.0 0.0 0.0

File: src/scene/model/xacro/sensor-camera.xacro (robot description, xacro)
@@ -2,5 +2,5 @@
   <gazebo reference="camera">
     <sensor type="camera" name="camera_node">
-      <update_rate>30.0</update_rate>
+      <update_rate>10.0</update_rate>
       <camera name="head">
         <horizontal_fov>1.3962634</horizontal_fov>
@@ -39,5 +39,5 @@
     <plugin name="camera_pose" filename="libgazebo_ros_p3d.so">
       <alwaysOn>true</alwaysOn>
-      <updateRate>50.0</updateRate>
+      <updateRate>10.0</updateRate>
       <bodyName>camera</bodyName>
       <topicName>camera_ground_truth</topicName>

File: src/scene/model/xacro/sensor-imu.xacro (robot description, xacro)
@@ -5,5 +5,5 @@
     <sensor name="imu_sensor" type="imu">
       <always_on>true</always_on>
-      <update_rate>400</update_rate>
+      <update_rate>400.0</update_rate>
       <visualize>true</visualize>
       <topic>__default_topic__</topic>
@@ -11,5 +11,5 @@
         <topicName>/sim_imu/frame</topicName>
         <bodyName>imu</bodyName>
-        <updateRateHZ>400</updateRateHZ>
+        <updateRateHZ>400.0</updateRateHZ>
         <gaussianNoise>0.0</gaussianNoise>
         <xyzOffset>0 0 0</xyzOffset>
@@ -24,5 +24,5 @@
     <plugin name="imu_pose" filename="libgazebo_ros_p3d.so">
       <alwaysOn>true</alwaysOn>
-      <updateRate>50.0</updateRate>
+      <updateRate>400.0</updateRate>
       <bodyName>imu</bodyName>
       <topicName>imu_ground_truth</topicName>

File: src/scene/model/xacro/sim-robot.xacro (robot description, xacro)
@@ -1,10 +1,10 @@
 <robot xmlns:xacro="http://www.ros.org/wiki/xacro" name="sim-robot">
   <xacro:property name="foot_box_size" value="0.001" />
-  <xacro:property name="base_box_size" value="0.3" />
+  <xacro:property name="base_box_size" value="0.1" />
   <xacro:property name="imu_box_size" value="0.06" />
   <xacro:property name="lidar_cylinder_radius" value="0.05" />
   <xacro:property name="lidar_cylinder_length" value="0.05" />
   <xacro:property name="arm_cylinder_radius" value="0.01" />
-  <xacro:property name="arm_cylinder_length" value="0.1" />
+  <xacro:property name="arm_cylinder_length" value="0.05" />
   <xacro:property name="wheel_cylinder_radius" value="0.08" />
   <xacro:property name="wheel_cylinder_length" value="0.04" />
@@ -79,8 +79,8 @@
   <xacro:include filename="imu.xacro" />
   <xacro:include filename="camera.xacro" />
-  <xacro:include filename="sensor-laser.xacro" />
+  <xacro:include filename="sensor-lidar.xacro" />
   <xacro:include filename="sensor-imu.xacro" />
   <xacro:include filename="sensor-camera.xacro" />
-  <xacro:include filename="wheels.xacro" />
-  <xacro:include filename="motion.xacro" />
+  <!-- <xacro:include filename="wheels.xacro" /> -->
+  <!-- <xacro:include filename="motion.xacro" /> -->
 </robot>

Commit message: update

File: src/scene/model/urdf/sim-robot.urdf (robot description, URDF)
Before this commit: robot sim-robot, 6 links, 5 joints
Joints:
- joint camera_to_base_link: origin xyz=0.08 0.0 0.0 rpy=0.0 0.0 0.0 -> xyz=0.08 0.0 0.0 rpy=0.0 1.57079632675 0.0

File: src/scene/model/xacro/camera.xacro (robot description, xacro)
@@ -23,5 +23,5 @@
     <parent link="base_link" />
     <child link="camera" />
-    <origin xyz="${base_box_size * 0.5 + camera_box_radius * 0.5} 0.0 0.0" rpy="0.0 0.0 0.0" />
+    <origin xyz="${base_box_size * 0.5 + camera_box_radius * 0.5} 0.0 0.0" rpy="0.0 ${PI * 0.5} 0.0" />
     <axis xyz="0.0 0.0 1.0" />
   </joint>

File: src/scene/model/xacro/sensor-camera.xacro (robot description, xacro)
@@ -22,5 +22,5 @@
       <plugin name="gazebo_camera" filename="libgazebo_ros_camera.so">
         <alwaysOn>true</alwaysOn>
-        <updateRate>0.0</updateRate>
+        <updateRate>10.0</updateRate>
         <cameraName>/sim_camera</cameraName>
         <imageTopicName>frame</imageTopicName>

File: src/scene/model/xacro/sensor-imu.xacro (robot description, xacro)
@@ -24,5 +24,5 @@
     <plugin name="imu_pose" filename="libgazebo_ros_p3d.so">
       <alwaysOn>true</alwaysOn>
-      <updateRate>1000.0</updateRate>
+      <updateRate>10.0</updateRate>
       <bodyName>imu</bodyName>
       <topicName>imu_ground_truth</topicName>

Commit message: update

File: src/scene/model/urdf/sim-robot.urdf (robot description, URDF)
Before this commit: robot sim-robot, 6 links, 5 joints
Joints:
- joint camera_to_base_link: origin xyz=0.08 0.0 0.0 rpy=0.0 1.57079632675 0.0 -> xyz=0.08 0.0 0.0 rpy=-1.57079632675 0.0 -1.57079632675

File: src/scene/model/xacro/camera.xacro (robot description, xacro)
@@ -23,5 +23,5 @@
     <parent link="base_link" />
     <child link="camera" />
-    <origin xyz="${base_box_size * 0.5 + camera_box_radius * 0.5} 0.0 0.0" rpy="0.0 ${PI * 0.5} 0.0" />
+    <origin xyz="${base_box_size * 0.5 + camera_box_radius * 0.5} 0.0 0.0" rpy="${PI * -0.5} 0.0 ${PI * -0.5}" />
     <axis xyz="0.0 0.0 1.0" />
   </joint>

Commit message: update[gen sim traj]

File: src/scene/model/urdf/sim-robot.urdf (robot description, URDF)
Before this commit: robot sim-robot, 6 links, 5 joints
Joints:
- joint camera_to_base_link: origin xyz=0.08 0.0 0.0 rpy=-1.57079632675 0.0 -1.57079632675 -> xyz=0.08 0.0 0.0 rpy=-1.57079632675 -0.785398163375 -1.57079632675

File: src/scene/model/xacro/camera.xacro (robot description, xacro)
@@ -23,5 +23,5 @@
     <parent link="base_link" />
     <child link="camera" />
-    <origin xyz="${base_box_size * 0.5 + camera_box_radius * 0.5} 0.0 0.0" rpy="${PI * -0.5} 0.0 ${PI * -0.5}" />
+    <origin xyz="${base_box_size * 0.5 + camera_box_radius * 0.5} 0.0 0.0" rpy="${PI * -0.5} ${PI * -0.25} ${PI * -0.5}" />
     <axis xyz="0.0 0.0 1.0" />
   </joint>
